File: rollo control.kicad_pcb (KiCad board)
At the start: 2 copper layers, 54 parts, among them IC1 IFX007TAUMA1, IC2 IFX007TAUMA1, IC3 BD63620AEFV, J2 Conn_01x02, J3 Conn_01x02, J4 Conn_01x02, K1 TIANBO-HJR-4102-L, K2 TIANBO-HJR-4102-L, K3 TIANBO-HJR-4102-L, U1 AP63205WU, U2 AP7384-33SA, U3 MAX485E

Commit message: place
Parts:
- removed C21: 1n, Capacitor_SMD:C_0603_1608Metric_Pad1.08x0.95mm_HandSolder
- removed CON_1, J3, J4: Conn_01x02, Connector_Phoenix_MSTB:PhoenixContact_MSTBA_2,5_2-G-5,08_1x02_P5.08mm_Horizontal
- removed IC3: BD63620AEFV, extlib:SOP65P760X100-24N
- removed the R27 at (78.7, 94.4)
- removed the R28 at (84.0, 94.4)
- added C15: 10n, Capacitor_SMD:C_0603_1608Metric_Pad1.08x0.95mm_HandSolder, F.Cu at (176.4, 74.4)
- added C17: 470uF, Capacitor_THT:C_Radial_D10.0mm_H16.0mm_P5.00mm, F.Cu at (203.5, 98.0)
- added C26: 1u, Capacitor_SMD:C_0603_1608Metric_Pad1.08x0.95mm_HandSolder, F.Cu at (157.6, 77.1)
- added C27: 1u, Capacitor_SMD:C_0603_1608Metric_Pad1.08x0.95mm_HandSolder, F.Cu at (157.6, 79.6)
- added C28: 1u, Capacitor_SMD:C_0603_1608Metric_Pad1.08x0.95mm_HandSolder, F.Cu at (157.6, 82.2)
- added C29: C_Small, Capacitor_SMD:C_0603_1608Metric_Pad1.08x0.95mm_HandSolder, F.Cu at (157.6, 84.7)
- added C30: C_Small, Capacitor_SMD:C_0603_1608Metric_Pad1.08x0.95mm_HandSolder, F.Cu at (157.6, 87.2)
- added CON_485_IN1: Conn_01x04, Connector_Phoenix_MC:PhoenixContact_MC_1,5_4-G-3.81_1x04_P3.81mm_Horizontal, F.Cu at (132.6, 72.2)
- added CON_485_OUT1: Conn_01x04, Connector_Phoenix_MC:PhoenixContact_MC_1,5_4-G-3.81_1x04_P3.81mm_Horizontal, F.Cu at (132.6, 90.2)
- added CON_NTC1: Conn_01x02, Connector_Phoenix_MSTB:PhoenixContact_MSTBA_2,5_2-G-5,08_1x02_P5.08mm_Horizontal, F.Cu at (64.0, 132.7)
- added CON_STEPPER1: Conn_01x04, Connector_JST:JST_XH_S4B-XH-A_1x04_P2.50mm_Horizontal, F.Cu at (76.5, 133.5)
- added D10: SP0502BAHT, Package_TO_SOT_SMD:SOT-23, F.Cu at (176.6, 96.9)
- added D11: SP0502BAHT, Package_TO_SOT_SMD:SOT-23, F.Cu at (186.5, 101.1)
- added D2: SP0502BAHT, Package_TO_SOT_SMD:SOT-23, F.Cu at (165.4, 69.5)
- added D5: SP0502BAHT, Package_TO_SOT_SMD:SOT-23, F.Cu at (165.4, 74.0)
- added D6: BZV55C3V6, Diode_SMD:D_MiniMELF, F.Cu at (171.1, 69.0)
- added D7: BAV70S, Package_TO_SOT_SMD:SOT-363_SC-70-6, F.Cu at (165.1, 96.6)
- added D8: BAV70S, Package_TO_SOT_SMD:SOT-363_SC-70-6, F.Cu at (165.1, 100.4)
- added DCDRIVE1: Conn_01x02, Connector_Phoenix_MSTB:PhoenixContact_MSTBA_2,5_2-G-5,08_1x02_P5.08mm_Horizontal, F.Cu at (91.5, 133.2)
- added FLOW_CON2: Conn_01x03, Connector_Phoenix_MSTB:PhoenixContact_MSTBA_2,5_3-G_1x03_P5.00mm_Horizontal, F.Cu at (52.3, 101.5)
- added PWR_IN2: Conn_01x02, Connector_Phoenix_MSTB:PhoenixContact_MSTBA_2,5_2-G-5,08_1x02_P5.08mm_Horizontal, F.Cu at (118.0, 54.3)
- added R22: 10k, Resistor_SMD:R_0805_2012Metric_Pad1.20x1.40mm_HandSolder, F.Cu at (176.6, 68.8)
- added R23: 22k, Resistor_SMD:R_0805_2012Metric_Pad1.20x1.40mm_HandSolder, F.Cu at (176.6, 71.7)
- added R30: 10k, Resistor_SMD:R_0805_2012Metric_Pad1.20x1.40mm_HandSolder, F.Cu at (153.0, 80.3)
- added R31: 10k, Resistor_SMD:R_0805_2012Metric_Pad1.20x1.40mm_HandSolder, F.Cu at (153.0, 83.2)
- added R32: 10k, Resistor_SMD:R_0805_2012Metric_Pad1.20x1.40mm_HandSolder, F.Cu at (153.0, 86.2)
- added R33: R_Small, Resistor_SMD:R_0805_2012Metric_Pad1.20x1.40mm_HandSolder, F.Cu at (153.0, 89.2)
- added R34: R_Small, Resistor_SMD:R_0805_2012Metric_Pad1.20x1.40mm_HandSolder, F.Cu at (153.0, 92.1)
- added R35: R_Small, Resistor_SMD:R_0805_2012Metric_Pad1.20x1.40mm_HandSolder, F.Cu at (153.0, 95.0)
- added R36: R_Small, Resistor_SMD:R_0805_2012Metric_Pad1.20x1.40mm_HandSolder, F.Cu at (153.0, 98.0)
- added U1: STM32G071RBTx, Package_QFP:LQFP-64_10x10mm_P0.5mm, B.Cu at (64.5, 68.5)
- added U4: AP7384-50SA, Package_TO_SOT_SMD:SOT-23, F.Cu at (169.7, 96.9)
- added U6: ULN2004A, Package_SO:TSSOP-16_4.4x5mm_P0.65mm, F.Cu at (188.4, 70.6)
- added U7: BTS724G, Package_SO:Infineon_PG-DSO-20-32, F.Cu at (206.7, 83.0)
- added U8: TXB0104PW, Package_SO:TSSOP-14_4.4x5mm_P0.65mm, F.Cu at (188.4, 95.6)
- added VIC_EN2: Conn_01x02, Connector_Phoenix_MSTB:PhoenixContact_MSTBA_2,5_2-G-5,08_1x02_P5.08mm_Horizontal, F.Cu at (77.5, 54.0)
- added VIC_EN3: Conn_01x02, Connector_Phoenix_MSTB:PhoenixContact_MSTBA_2,5_2-G-5,08_1x02_P5.08mm_Horizontal, F.Cu at (91.0, 54.3)
- I2C_CON1: footprint Connector_JST:JST_XH_B5B-XH-A_1x05_P2.50mm_Vertical -> Connector_JST:JST_XH_B4B-XH-A_1x04_P2.50mm_Vertical
- IC2: footprint extlib:PG-TO263-7-1 -> kicad_customlib:PG-TO263-7-1
- R17: renamed from R21; value 10meg -> 10k
- R18: renamed from R20; value 10meg -> 10k
- R29: value 39k -> 10k
- moved I2C_CON1 85.2 mm to (121.0, 138.0)
- moved R29 77.7 mm to (153.0, 77.3)
- moved PWR_IN1 52.9 mm to (104.5, 54.3), turned to 180 degrees
- moved VIC_EN1 48.8 mm to (64.0, 54.3), turned to 180 degrees
- moved D4 41.0 mm to (114.5, 105.0)
- moved D1 41.0 mm to (114.5, 98.3)
- moved D3 41.0 mm to (114.5, 101.7)
- moved U5 39.7 mm to (91.5, 116.0)
- moved C4 36.8 mm to (80.5, 102.5)
- moved EXT_REL_CON1 33.2 mm to (104.5, 138.0)
- moved IC1 31.5 mm to (93.0, 84.0)
- moved IC2 31.5 mm to (105.0, 84.0)
- moved D9 29.2 mm to (109.4, 115.0)
- moved ONE_CON1 26.7 mm to (45.5, 132.7)
- moved A1 22.2 mm to (63.2, 86.6)
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- renumbered C23 to C16, C20 to C25, C8 to C4, D2 to D1, D1 to D9, R9 to R10, R16 to R11, R10 to R12, R17 to R13, R11 to R14, R12 to R15, R19 to R16, R13 to R19, R18 to R20, R14 to R21, R22 to R24, R23 to R25, R24 to R26, R25 to R27, R26 to R28, R15 to R9, U1 to U2, U2 to U3, U3 to U5, J2 to VIC_EN1
Connections:
- net /Digital In/BTN_1 renamed BTN_1
- net /Digital In/BTN_2 renamed BTN_2
- net /Digital In/FLW_SIG renamed FLW_Sig1
- net /Digital In/ONE_SIG renamed ONE_SIG
- net /Modbus/485_enable renamed enable
- net /Modbus/485_pico renamed pico
- net /Modbus/485_poci renamed poci
- net /Stepper/MS1 renamed Step_MS1
- net /Stepper/MS2 renamed Step_MS2
- net /Stepper/MS3 renamed Step_MS3
- net /Stepper/dir renamed Step_dir
- net /Stepper/enable renamed Step_enable
- net /Stepper/reset renamed Step_reset
- net /Stepper/sleep renamed Step_sleep
- net /Stepper/step renamed Step_step
- A1 pad 1: /Stepper/GND -> /Batt-
- A1 pad 2: /Stepper/3V3 -> /Autoterm/3V3
- A1 pad 7: /Stepper/GND -> /Batt-
- BTN_1 pad 1: /Digital In/5V -> /DC Power/5V0
- BTN_1 pad 3: /Digital In/GND -> /GND
- BTN_2 pad 1: /Digital In/5V -> /DC Power/5V0
- BTN_2 pad 3: /Digital In/GND -> /GND
- C12 pad 2: /Digital In/GND -> /GND
- C13 pad 2: /Digital In/GND -> /GND
- C14 pad 2: /Digital In/GND -> /GND
- C16 pad 2: /Stepper/GND -> /Batt-
- C25 pad 1: /Modbus/5V0 -> /DC Power/5V0
- C25 pad 2: /Modbus/GND -> /GND
- C4 pad 1: /DC Drive/VS -> /12V0
- C4 pad 2: /DC Drive/GND -> /Batt-
- D1 pad 2: /Digital In/GND -> /GND
- D3 pad 2: /Digital In/GND -> /GND
- D4 pad 2: /Digital In/GND -> /GND
- D9 pad 3: /Modbus/GND -> /GND
- EXT_REL_CON1 pad 1: /mcu relais/5V0 -> /DC Power/5V0
- FLOW_CON1 pad 1: /Digital In/5V -> /DC Power/5V0
- FLOW_CON1 pad 3: /Digital In/GND -> /GND
- I2C_CON1 pad 2: /Digital In/GND -> /GND
- I2C_CON1 pad 3: /Digital In/I2C_SCL -> I2C_SCL
- I2C_CON1 pad 4: /Digital In/I2C_SDA -> I2C_SDA
- IC1 pad 1: /DC Drive/GND -> /Batt-
- IC1 pad 4: /DC Drive/DC+ -> Net-(DCDRIVE1-Pin_1)
- IC1 pad 7: /DC Drive/VS -> Net-(IC1-VS)
- IC1 pad 8: /DC Drive/DC- -> Net-(DCDRIVE1-Pin_1)
- IC2 pad 1: /DC Drive/GND -> /Batt-
- IC2 pad 4: /DC Drive/DC+ -> Net-(DCDRIVE1-Pin_2)
- IC2 pad 7: /DC Drive/VS -> Net-(IC1-VS)
- IC2 pad 8: /DC Drive/DC+ -> Net-(DCDRIVE1-Pin_2)
- K1 pad 8: /mcu relais/5V0 -> /DC Power/5V0
- K2 pad 8: /mcu relais/5V0 -> /DC Power/5V0
- K3 pad 8: /mcu relais/5V0 -> /DC Power/5V0
- ONE_CON1 pad 3: /Digital In/GND -> /GND
- PWR_IN1 pad 1: /DC Power/GND -> /Batt-
- PWR_IN1 pad 2: Net-(PWR_IN1-Pin_2) -> /12V0
- R11 pad 1: /Digital In/3V3 -> /Autoterm/3V3
- R12 pad 1: /Digital In/GND -> /GND
- R13 pad 1: /Digital In/3V3 -> /Autoterm/3V3
- R15 pad 1: /Digital In/GND -> /GND
- R16 pad 1: /Digital In/3V3 -> /Autoterm/3V3
- R17 pad 1: /Digital In/3V3 -> /Autoterm/3V3
- R17 pad 2: /Digital In/I2C_SDA -> I2C_SCL
- R18 pad 1: /Digital In/3V3 -> /Autoterm/3V3
- R18 pad 2: /Digital In/I2C_SCL -> I2C_SDA
- R20 pad 1: /Digital In/5V -> /DC Power/5V0
- R21 pad 1: /Digital In/GND -> /GND
- R24 pad 2: /Modbus/5V0 -> /DC Power/5V0
- R28 pad 1: /Modbus/GND -> /GND
- R29 pad 1: Net-(IC3-CR) -> /Analog-IN/5V0
- R29 pad 2: /Stepper/GND -> Net-(CON_NTC1-Pin_1)
- R9 pad 1: /Digital In/5V -> /DC Power/5V0
- U2 pad 2: Net-(PWR_IN1-Pin_2) -> Net-(D8A-K)
- U2 pad 3: Net-(PWR_IN1-Pin_2) -> Net-(D8A-K)
- U2 pad 4: /DC Power/GND -> /Batt-
- U3 pad 2: /DC Power/3V3 -> /Autoterm/3V3
- U3 pad 3: /DC Power/GND -> /Batt-
- U5 pad 5: /Modbus/GND -> /GND
- U5 pad 8: /Modbus/5V0 -> /DC Power/5V0
Other:
- board outline added: 100 x 100 mm
- copper layers 2 -> 4

Commit message: 605
Parts:
- added C34: 1u, Capacitor_SMD:C_0603_1608Metric_Pad1.08x0.95mm_HandSolder, F.Cu at (187.9, 126.9)
- added C35: 1u, Capacitor_SMD:C_0603_1608Metric_Pad1.08x0.95mm_HandSolder, F.Cu at (187.9, 129.4)
- added C36: 1u, Capacitor_SMD:C_0603_1608Metric_Pad1.08x0.95mm_HandSolder, F.Cu at (187.9, 131.9)
- added CON_NTC2: Conn_01x02, Connector_Phoenix_MC:PhoenixContact_MC_1,5_2-G-3.5_1x02_P3.50mm_Horizontal, F.Cu at (146.2, 148.2)
- added CON_PUMP1: Conn_01x02, Connector_Phoenix_MC:PhoenixContact_MC_1,5_2-G-3.5_1x02_P3.50mm_Horizontal, F.Cu at (162.9, 116.6)
- added CON_PUMP2: Conn_01x02, Connector_Phoenix_MC:PhoenixContact_MC_1,5_2-G-3.5_1x02_P3.50mm_Horizontal, F.Cu at (146.2, 134.1)
- added CON_PUMP3: Conn_01x02, Connector_Phoenix_MC:PhoenixContact_MC_1,5_2-G-3.5_1x02_P3.50mm_Horizontal, F.Cu at (156.7, 134.1)
- added CON_PUMP4: Conn_01x02, Connector_Phoenix_MC:PhoenixContact_MC_1,5_2-G-3.5_1x02_P3.50mm_Horizontal, F.Cu at (167.3, 134.1)
- added D12: SP0502BAHT, Package_TO_SOT_SMD:SOT-23, F.Cu at (192.6, 127.8)
- added D13: BZV55B5V6, Diode_SMD:D_MiniMELF, F.Cu at (157.2, 52.2)
- added D14: BZV55B5V6, Diode_SMD:D_MiniMELF, F.Cu at (157.2, 55.6)
- added D15: BZV55B3V6, Diode_SMD:D_MiniMELF, F.Cu at (157.2, 58.9)
- added F1: Fuse_Small, Fuse:Fuse_1210_3225Metric_Pad1.42x2.65mm_HandSolder, F.Cu at (163.4, 52.6)
- added F2: Fuse, Fuse:Fuseholder_Blade_ATO_Littelfuse_Pudenz_2_Pin, F.Cu at (154.9, 43.8)
- added JP10: Jumper_3_Bridged12, Connector_PinHeader_2.54mm:PinHeader_1x03_P2.54mm_Vertical, F.Cu at (183.3, 155.9)
- added JP6: Jumper_3_Bridged12, Connector_PinHeader_2.54mm:PinHeader_1x03_P2.54mm_Vertical, F.Cu at (176.7, 115.8)
- added JP7: Jumper_3_Bridged12, Connector_PinHeader_2.54mm:PinHeader_1x03_P2.54mm_Vertical, F.Cu at (190.0, 155.9)
- added ONE_CON2: Conn_01x03, Connector_Phoenix_MC:PhoenixContact_MC_1,5_3-G-3.5_1x03_P3.50mm_Horizontal, F.Cu at (184.6, 142.6)
- added R1: R, Resistor_SMD:R_0201_0603Metric_Pad0.64x0.40mm_HandSolder, F.Cu at (169.7, 51.4)
- added R2: R, Resistor_SMD:R_0201_0603Metric_Pad0.64x0.40mm_HandSolder, F.Cu at (169.7, 53.2)
- added R3: R, Resistor_SMD:R_0201_0603Metric_Pad0.64x0.40mm_HandSolder, F.Cu at (169.7, 54.9)
- added R30: 10k, Resistor_SMD:R_0201_0603Metric_Pad0.64x0.40mm_HandSolder, F.Cu at (174.6, 53.2)
- added R31: 10k, Resistor_SMD:R_0201_0603Metric_Pad0.64x0.40mm_HandSolder, F.Cu at (174.6, 54.9)
- added R32: 10k, Resistor_SMD:R_0201_0603Metric_Pad0.64x0.40mm_HandSolder, F.Cu at (174.6, 56.7)
- added R33: ~, Resistor_SMD:R_0201_0603Metric_Pad0.64x0.40mm_HandSolder, F.Cu at (174.6, 58.4)
- added R34: ~, Resistor_SMD:R_0201_0603Metric_Pad0.64x0.40mm_HandSolder, F.Cu at (174.6, 60.2)
- added R35: ~, Resistor_SMD:R_0201_0603Metric_Pad0.64x0.40mm_HandSolder, F.Cu at (177.4, 51.4)
- added R36: ~, Resistor_SMD:R_0201_0603Metric_Pad0.64x0.40mm_HandSolder, F.Cu at (177.4, 53.2)
- added R37: 10k, Resistor_SMD:R_0805_2012Metric_Pad1.20x1.40mm_HandSolder, F.Cu at (183.4, 127.1)
- added R37: 10k, Resistor_SMD:R_0201_0603Metric_Pad0.64x0.40mm_HandSolder, F.Cu at (177.4, 54.9)
- added R38: 10k, Resistor_SMD:R_0805_2012Metric_Pad1.20x1.40mm_HandSolder, F.Cu at (183.4, 130.0)
- added R38: 10k, Resistor_SMD:R_0201_0603Metric_Pad0.64x0.40mm_HandSolder, F.Cu at (177.4, 56.7)
- added R39: 10k, Resistor_SMD:R_0201_0603Metric_Pad0.64x0.40mm_HandSolder, F.Cu at (177.4, 58.4)
- added R39: 10k, Resistor_SMD:R_0805_2012Metric_Pad1.20x1.40mm_HandSolder, F.Cu at (183.4, 133.0)
- added R4: R, Resistor_SMD:R_0201_0603Metric_Pad0.64x0.40mm_HandSolder, F.Cu at (169.7, 56.7)
- added R40: 10k, Resistor_SMD:R_0805_2012Metric_Pad1.20x1.40mm_HandSolder, F.Cu at (183.4, 135.9)
- added R5: R, Resistor_SMD:R_0201_0603Metric_Pad0.64x0.40mm_HandSolder, F.Cu at (169.7, 58.4)
- added R6: R, Resistor_SMD:R_0201_0603Metric_Pad0.64x0.40mm_HandSolder, F.Cu at (169.7, 60.2)
- added R7: R, Resistor_SMD:R_0201_0603Metric_Pad0.64x0.40mm_HandSolder, F.Cu at (169.7, 61.9)
- added R8: 10k, Resistor_SMD:R_0201_0603Metric_Pad0.64x0.40mm_HandSolder, F.Cu at (174.6, 51.4)
- BTN_1, BTN_2, FLOW_CON1, FLOW_CON2, ONE_CON1: footprint Connector_Phoenix_MSTB:PhoenixContact_MSTBA_2,5_3-G_1x03_P5.00mm_Horizontal -> Connector_Phoenix_MC:PhoenixContact_MC_1,5_3-G-3.5_1x03_P3.50mm_Horizontal
- CON_485_IN1, CON_485_OUT1: footprint Connector_Phoenix_MC:PhoenixContact_MC_1,5_4-G-3.81_1x04_P3.81mm_Horizontal -> Connector_Phoenix_MC:PhoenixContact_MC_1,5_4-G-3.5_1x04_P3.50mm_Horizontal
- CON_NTC1: footprint Connector_Phoenix_MSTB:PhoenixContact_MSTBA_2,5_2-G-5,08_1x02_P5.08mm_Horizontal -> Connector_Phoenix_MC:PhoenixContact_MC_1,5_2-G-3.5_1x02_P3.50mm_Horizontal
- CON_STEPPER1: footprint Connector_JST:JST_XH_S4B-XH-A_1x04_P2.50mm_Horizontal -> Connector_Phoenix_MC:PhoenixContact_MC_1,5_4-G-3.5_1x04_P3.50mm_Horizontal
- R10, R11, R12, R13, R14, R15, R16, R17, R18, R19, R20, R21, R22, R23, R24, R25, R26, R27, R28, R29, R9: footprint Resistor_SMD:R_0805_2012Metric_Pad1.20x1.40mm_HandSolder -> Resistor_SMD:R_0201_0603Metric_Pad0.64x0.40mm_HandSolder
Connections:
- net Ain_ntc+ renamed Ain_ntc0+
- net Ain_ntc- renamed Ain_ntc0-
- BTN_1 pad 1: /DC Power/5V0 -> /Autoterm/5V0
- BTN_2 pad 1: /DC Power/5V0 -> /Autoterm/5V0
- C25 pad 1: /DC Power/5V0 -> /Autoterm/5V0
- C28 pad 2: /GND -> /Analog-IN/GND
- C29 pad 2: /GND -> /Analog-IN/GND
- C30 pad 2: /GND -> /Analog-IN/GND
- CON_485_IN1 pad 1: /DC Power/5V0 -> /Autoterm/5V0
- CON_485_OUT1 pad 1: /DC Power/5V0 -> /Autoterm/5V0
- D10 pad 3: /GND -> /Analog-IN/GND
- D7 pad 6: /DC Power/5V0 -> /Autoterm/5V0
- EXT_REL_CON1 pad 1: /DC Power/5V0 -> Net-(EXT_REL_CON1-Pin_1)
- FLOW_CON1 pad 1: /DC Power/5V0 -> /Autoterm/5V0
- FLOW_CON2 pad 1: /DC Power/5V0 -> /Autoterm/5V0
- K1 pad 8: /DC Power/5V0 -> Net-(EXT_REL_CON1-Pin_1)
- K2 pad 8: /DC Power/5V0 -> Net-(EXT_REL_CON1-Pin_1)
- K3 pad 8: /DC Power/5V0 -> Net-(EXT_REL_CON1-Pin_1)
- L1 pad 2: /DC Power/5V0 -> /Autoterm/5V0
- PWR_IN1 pad 2: /12V0 -> Net-(PWR_IN1-Pin_2)
- PWR_IN2 pad 2: /24V0 -> Net-(PWR_IN2-Pin_2)
- R20 pad 1: /DC Power/5V0 -> /Autoterm/5V0
- R24 pad 2: /DC Power/5V0 -> /Autoterm/5V0
- R32 pad 1: /GND -> /Analog-IN/GND
- R35 pad 2: /GND -> /Analog-IN/GND
- R36 pad 2: /GND -> /Analog-IN/GND
- R9 pad 1: /DC Power/5V0 -> /Autoterm/5V0
- U2 pad 1: /DC Power/5V0 -> /Autoterm/5V0
- U2 pad 2: Net-(D8A-K) -> Net-(U2-EN)
- U2 pad 3: Net-(D8A-K) -> Net-(U2-EN)
- U3 pad 1: /DC Power/5V0 -> /Autoterm/5V0
- U4 pad 1: Net-(D8A-K) -> Net-(U2-EN)
- U5 pad 8: /DC Power/5V0 -> /Autoterm/5V0
- U6 pad 9: /DC Power/5V0 -> Net-(EXT_REL_CON1-Pin_1)
