File: rollo control.kicad_pcb (KiCad board)
At the start: 4 copper layers, 100 x 100 mm, 152 parts, among them IC1 IFX007TAUMA1, IC2 IFX007TAUMA1, K1 TIANBO-HJR-4102-L, K2 TIANBO-HJR-4102-L, K3 TIANBO-HJR-4102-L, U1 STM32G071RBTx, U2 AP63205WU, U3 AP7384-33SA, U4 AP7384-50SA, U5 MAX485E, U6 ULN2004A, U7 BTS724G, U8 TXB0104PW

Commit message: asdf
Parts:
- U6: moved to B.Cu
- moved ONE_CON1 112.3 mm to (123.6, 134.9), turned to 0 degrees
- moved CON_485_OUT1 98.1 mm to (50.6, 107.8), turned to -90 degrees
- moved ONE_CON2 93.7 mm to (110.2, 134.9), turned to 0 degrees
- moved FLOW_CON2 75.3 mm to (96.9, 134.9), turned to 0 degrees
- moved CON_485_IN1 72.6 mm to (50.6, 124.3), turned to -90 degrees
- moved FLOW_CON1 57.1 mm to (83.5, 134.9), turned to 0 degrees
- moved R20 48.6 mm to (74.0, 141.1), turned to 90 degrees
- moved D1 45.8 mm to (-5.24, 118.4)
- moved D3 45.8 mm to (-5.24, 121.8)
- moved D4 45.8 mm to (-5.24, 125.1)
- moved R13 45.1 mm to (71.0, 141.1), turned to 90 degrees
- moved K1 45.0 mm to (128.9, 97.8), turned to 180 degrees
- moved R11 41.8 mm to (68.1, 141.1), turned to 90 degrees
- moved BTN_2 39.6 mm to (70.2, 134.9), turned to 0 degrees
- moved U6 39.3 mm to (114.3, 92.7), turned to 180 degrees
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Routing:
- net (no net): vias 2 -> 4

Commit message: placing2
Parts:
- removed JP4, JP5: Jumper_2_Bridged, Connector_PinHeader_2.54mm:PinHeader_1x02_P2.54mm_Vertical
- removed JP7: Jumper_3_Bridged12, Connector_PinHeader_2.54mm:PinHeader_1x03_P2.54mm_Vertical
- removed the R30 at (174.6, 53.2)
- removed the R31 at (174.6, 54.9)
- removed the R32 at (174.6, 56.7)
- removed the R37 at (183.4, 127.1)
- removed the R38 at (177.4, 56.7)
- removed the R39 at (183.4, 133.0)
- C12, C26, C27, C28, C31, C32, C34, C35, C36, D1, D10, D11, D12, D2, JP10, R10, R11, R12, R13, R29, R37, R39, R8, R9, U8: moved to B.Cu
- D7: footprint Package_TO_SOT_SMD:SOT-363_SC-70-6 -> Package_TO_SOT_SMD:SOT-323_SC-70_Handsoldering
- R30, R31, R32, R38: footprint Resistor_SMD:R_0805_2012Metric_Pad1.20x1.40mm_HandSolder -> Resistor_SMD:R_0201_0603Metric_Pad0.64x0.40mm_HandSolder; moved to B.Cu
- R33, R34, R35, R36: value R_Small -> ~; footprint Resistor_SMD:R_0805_2012Metric_Pad1.20x1.40mm_HandSolder -> Resistor_SMD:R_0201_0603Metric_Pad0.64x0.40mm_HandSolder
- moved I2C_CON1 104.0 mm to (110.5, 123.3), turned to 180 degrees
- moved UART_AUTOTERM1 102.1 mm to (110.5, 115.5), turned to 180 degrees
- moved U8 95.0 mm to (96.0, 117.8), turned to 180 degrees
- moved D11 92.9 mm to (94.2, 112.5), turned to 180 degrees
- moved R8 88.9 mm to (126.2, 126.1)
- moved R35 82.0 mm to (216.8, 123.3)
- moved R36 82.0 mm to (216.8, 125.1)
- moved R33 81.7 mm to (216.8, 128.4)
- moved R34 81.7 mm to (216.8, 130.1)
- moved D2 81.4 mm to (111.0, 130.1), turned to 180 degrees
- moved D1 80.3 mm to (74.2, 129.5), turned to 180 degrees
- moved R37 76.2 mm to (125.4, 110.6)
- moved D12 73.9 mm to (120.4, 112.1), turned to -90 degrees
- moved R39 72.2 mm to (125.4, 108.6)
- moved C35 69.8 mm to (121.4, 108.3), turned to 90 degrees
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Connections:
- C36 pad 2: Net-(D12-A) -> /GND
- D12 pad 3: Net-(D12-A) -> /GND
- EXT_REL_CON1 pad 1: Net-(EXT_REL_CON1-Pin_1) -> /Autoterm/5V0
- K1 pad 8: Net-(EXT_REL_CON1-Pin_1) -> /Autoterm/5V0
- K2 pad 8: Net-(EXT_REL_CON1-Pin_1) -> /Autoterm/5V0
- K3 pad 8: Net-(EXT_REL_CON1-Pin_1) -> /Autoterm/5V0
- R30 pad 1: Ain_ntc0+ -> Ain_ntc0-
- R30 pad 2: Net-(CON_NTC1-Pin_1) -> Net-(CON_NTC1-Pin_2)
- R31 pad 1: Ain_ntc0- -> /GND
- R32 pad 1: /Analog-IN/GND -> /Analog-IN/5V0
- R32 pad 2: Net-(CON_NTC1-Pin_2) -> Net-(CON_NTC2-Pin_1)
- R33 pad 1: /12V0 -> Ain_24V_Sig
- R33 pad 2: Ain_24V_Sig -> /12V0
- R34 pad 1: /24V0 -> Ain_12V_Sig
- R34 pad 2: Ain_12V_Sig -> /24V0
- R35 pad 1: Ain_24V_Sig -> /GND
- R35 pad 2: /Analog-IN/GND -> Ain_12V_Sig
- R36 pad 1: Ain_12V_Sig -> /GND
- R36 pad 2: /Analog-IN/GND -> Ain_24V_Sig
- R38 pad 1: Ain_ntc1+ -> Ain_ntc1-
- R38 pad 2: Net-(CON_NTC2-Pin_1) -> Net-(CON_NTC2-Pin_2)
- R39 pad 1: Net-(D12-A) -> /GND
- U6 pad 9: Net-(EXT_REL_CON1-Pin_1) -> /Autoterm/5V0
Routing:
- net /Autoterm/5V0: track 0.00 -> 201.0 mm
- net Net-(VIC_EN3-Pin_2): track 0.00 -> 42.6 mm
- net Net-(U6-O3): track 0.00 -> 37.1 mm
- net Net-(ONE_CON1-Pin_1): track 0.00 -> 25.1 mm
- net Net-(EXT_REL_CON1-Pin_2): track 0.00 -> 23.6 mm
- net Net-(EXT_REL_CON1-Pin_3): track 0.00 -> 21.2 mm
- net Net-(U6-O1): track 0.00 -> 20.5 mm
- net Net-(VIC_EN3-Pin_1): track 0.00 -> 20.3 mm
- net Net-(EXT_REL_CON1-Pin_4): track 0.00 -> 18.9 mm
- net Net-(CON_NTC2-Pin_2): track 0.00 -> 16.8 mm
- net Net-(EXT_REL_CON1-Pin_5): track 0.00 -> 16.6 mm
- net Net-(CON_NTC2-Pin_1): track 0.00 -> 15.0 mm
- net Net-(U6-O2): track 0.00 -> 14.2 mm
- net ONE_SIG: track 0.00 -> 9.75 mm
- net Ain_ntc1+: track 0.00 -> 9.42 mm
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
Commit message: ende
Parts:
- removed the D7 at (172.0, 113.0)
- removed D8: BAV70S, Package_TO_SOT_SMD:SOT-323_SC-70_Handsoldering
- removed the R33 at (212.3, 121.7)
- removed the R34 at (216.8, 130.1)
- removed the R35 at (212.3, 127.6)
- removed the R36 at (212.3, 130.6)
- added D16: BAV70, Package_TO_SOT_SMD:SOT-23, B.Cu at (93.9, 54.2)
- C1, C10, C11, C13, C14, C15, C16, C18, C19, C2, C20, C21, C22, C24, C25, C29, C3, C30, C37, C5, C6, C7, C8, C9, D13, D14, D15, D3, D4, D5, D6, D7, D9, F1, IC1, IC2, L1, U1, U2, U3, U4, U5, U7: moved to B.Cu
- R1, R14, R15, R16, R17, R18, R19, R2, R20, R21, R22, R23, R24, R25, R26, R27, R28, R3, R33, R34, R35, R36, R4, R40, R5, R6, R7: footprint Resistor_SMD:R_0201_0603Metric_Pad0.64x0.40mm_HandSolder -> Resistor_SMD:R_0805_2012Metric_Pad1.20x1.40mm_HandSolder; moved to B.Cu
- R10, R11, R12, R13, R29, R30, R31, R32, R37, R38, R39, R8, R9: footprint Resistor_SMD:R_0201_0603Metric_Pad0.64x0.40mm_HandSolder -> Resistor_SMD:R_0805_2012Metric_Pad1.20x1.40mm_HandSolder
- moved C30 145.8 mm to (76.0, 82.2), turned to 180 degrees
- moved C29 145.7 mm to (76.0, 80.0), turned to 180 degrees
- moved R35 145.7 mm to (76.2, 85.0)
- moved R36 144.2 mm to (79.5, 81.0), turned to 90 degrees
- moved R33 142.9 mm to (82.0, 81.0), turned to 90 degrees
- moved R34 137.4 mm to (80.8, 85.0)
- moved C21 111.1 mm to (72.2, 60.9)
- moved R22 97.2 mm to (100.5, 129.2), turned to -90 degrees
- moved C15 95.9 mm to (97.5, 129.0), turned to 90 degrees
- moved D4 94.7 mm to (89.5, 125.5), turned to 180 degrees
- moved C20 94.0 mm to (77.2, 58.5), turned to 180 degrees
- moved R23 93.0 mm to (103.5, 129.2), turned to 90 degrees
- moved C19 90.3 mm to (77.2, 61.1), turned to 180 degrees
- moved U4 89.9 mm to (85.0, 66.5), turned to 180 degrees
- moved D6 89.3 mm to (101.8, 125.2), turned to 180 degrees
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Connections:
- net /12V0 renamed /Analog-IN/12V0
- net /24V0 renamed /Analog-IN/24V0
Routing:
- net /Analog-IN/12V0: track 0.00 -> 172.7 mm
- net /Analog-IN/24V0: track 0.00 -> 155.4 mm
- net /GND: track 0.25 -> 117.0 mm, vias 0 -> 19
- net /Autoterm/5V0: track 201.0 -> 314.6 mm
- net Net-(PWR_IN12-Pin_2): track 0.00 -> 86.4 mm
- net Net-(PWR_IN24-Pin_2): track 0.00 -> 52.1 mm
- net Net-(JP6-C): track 0.00 -> 51.1 mm
- net Net-(VIC_EN2-Pin_2): track 0.00 -> 50.0 mm
- net Net-(CON_485_IN1-Pin_3): track 0.00 -> 39.5 mm
- net Net-(U2-EN): track 0.00 -> 36.0 mm
- net Net-(CON_485_IN1-Pin_2): track 0.00 -> 34.5 mm
- net Net-(A1-VMOT): track 0.00 -> 33.9 mm
- net Net-(VIC_EN1-Pin_2): track 0.00 -> 26.0 mm, vias 0 -> 2
- net Net-(ONE_CON1-Pin_1): track 25.1 -> 0.00 mm
- net Net-(JP10-C): track 0.00 -> 23.0 mm
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- added copper zone on In2.Cu, net /GND
- added copper zone on B.Cu, net Net-(JP6-C)
