File: rollo control.kicad_pcb (KiCad board)
At the start: 4 copper layers, 100 x 100 mm, 143 parts, among them IC1 IFX007TAUMA1, IC2 IFX007TAUMA1, K1 TIANBO-HJR-4102-L, K2 TIANBO-HJR-4102-L, K3 TIANBO-HJR-4102-L, U1 STM32G071RBTx, U2 AP63205WU, U3 AP7384-33SA, U4 AP7384-50SA, U5 MAX485E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

Commit message: dgfg
Parts:
- removed A1: Pololu_Breakout_A4988, Module:Pololu_Breakout-16_15.2x20.3mm
- removed C16: 100n, Capacitor_SMD:C_0603_1608Metric_Pad1.08x0.95mm_HandSolder
- removed C17: 470uF, Capacitor_THT:C_Radial_D10.0mm_H16.0mm_P5.00mm
- removed CON_STEPPER1: Conn_01x04, Connector_Phoenix_MC:PhoenixContact_MC_1,5_4-G-3.5_1x04_P3.50mm_Horizontal
- removed JP1: Jumper_3_Bridged12, Connector_PinHeader_2.54mm:PinHeader_1x03_P2.54mm_Vertical

Commit message: gsdfg
dyfg
Parts:
- removed C30: C_Small, Capacitor_SMD:C_0603_1608Metric_Pad1.08x0.95mm_HandSolder
- removed D10, D11, D12: SP0502BAHT, Package_TO_SOT_SMD:SOT-23
- removed D8: BAV70S, Package_TO_SOT_SMD:SOT-323_SC-70_Handsoldering
- removed F1: Fuse_Small, Fuse:Fuse_1210_3225Metric_Pad1.42x2.65mm_HandSolder
- removed F3: Fuse, Fuse:Fuseholder_Clip-5x20mm_Littelfuse_100_Inline_P20.50x4.60mm_D1.30mm_Horizontal
- removed JP6, JP8: Jumper_3_Bridged12, Connector_PinHeader_2.54mm:PinHeader_1x03_P2.54mm_Vertical
- removed K1, K2, K3: TIANBO-HJR-4102-L, Relay_THT:Relay_SPDT_HJR-4102
- removed PWR_IN24, PWR_OUT24: Conn_01x02, Connector_Phoenix_MSTB:PhoenixContact_MSTBA_2,5_2-G-5,08_1x02_P5.08mm_Horizontal
- removed R34 (x2), R35 (x2): ~, Resistor_SMD:R_0201_0603Metric_Pad0.64x0.40mm_HandSolder
- removed VIC_EN1, VIC_EN2, VIC_EN3: Conn_01x02, Connector_Phoenix_MC:PhoenixContact_MC_1,5_2-G-3.5_1x02_P3.50mm_Horizontal
- added EXT_REL_CON2: Conn_01x06, Connector_JST:JST_XH_B5B-XH-A_1x05_P2.50mm_Vertical, F.Cu at (157.6, 104.1)
Connections:
- C2 pad 1: Net-(IC1-VS) -> /12V0
- C21 pad 1: Net-(U2-EN) -> /12V0
- C29 pad 1: Ain_24V_Sig -> Ain_12V_Sig
- C3 pad 1: Net-(IC1-VS) -> /12V0
- C37 pad 1: Net-(U2-EN) -> /12V0
- C4 pad 1: Net-(IC1-VS) -> /12V0
- C6 pad 1: Net-(IC1-VS) -> /12V0
- C9 pad 1: Net-(IC1-VS) -> /12V0
- IC1 pad 7: Net-(IC1-VS) -> /12V0
- IC2 pad 7: Net-(IC1-VS) -> /12V0
- R33 pad 1: Ain_24V_Sig -> Ain_12V_Sig (x2)
- R36 pad 2: Ain_24V_Sig -> Ain_12V_Sig (x2)
- U2 pad 2: Net-(U2-EN) -> /12V0
- U2 pad 3: Net-(U2-EN) -> /12V0
- U4 pad 1: Net-(U2-EN) -> /12V0
- U7 pad 1: Net-(JP6-C) -> /12V0
- U7 pad 10: Net-(JP6-C) -> /12V0
- U7 pad 11: Net-(JP6-C) -> /12V0
- U7 pad 12: Net-(JP6-C) -> /12V0
- U7 pad 15: Net-(JP6-C) -> /12V0
- U7 pad 16: Net-(JP6-C) -> /12V0
- U7 pad 19: Net-(JP6-C) -> /12V0
- U7 pad 20: Net-(JP6-C) -> /12V0
Routing:
- net (no net): track 0.00 -> 69.9 mm
- net Net-(VIC_EN3-Pin_2): track 42.6 -> 0.00 mm
- net Net-(VIC_EN3-Pin_1): track 20.3 -> 0.00 mm
- net Net-(VIC_EN1-Pin_1): track 7.07 -> 0.00 mm
