File: A4988Stepper.kicad_sch (KiCad schematic)
At the start: 6 parts

Commit message: place
Parts:
- CON_STEPPER1: footprint (none) -> Connector_JST:JST_XH_S4B-XH-A_1x04_P2.50mm_Horizontal
Changed lines of the file:
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@@
       (effects (font (size 1.27 1.27)) (justify left))
     )
-    (property "Footprint" "" (at 114.3 82.55 0)
+    (property "Footprint" "Connector_JST:JST_XH_S4B-XH-A_1x04_P2.50mm_Horizontal" (at 114.3 82.55 0)
       (effects (font (size 1.27 1.27)) hide)
     )

Commit message: mc1.5
Parts:
- CON_STEPPER1: footprint Connector_JST:JST_XH_S4B-XH-A_1x04_P2.50mm_Horizontal -> Connector_Phoenix_MC:PhoenixContact_MC_1,5_4-G-3.5_1x04_P3.50mm_Horizontal
Changed lines of the file:
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@@
       (effects (font (size 1.27 1.27)) (justify left))
     )
-    (property "Footprint" "Connector_JST:JST_XH_S4B-XH-A_1x04_P2.50mm_Horizontal" (at 114.3 82.55 0)
+    (property "Footprint" "Connector_Phoenix_MC:PhoenixContact_MC_1,5_4-G-3.5_1x04_P3.50mm_Horizontal" (at 114.3 82.55 0)
       (effects (font (size 1.27 1.27)) hide)
     )

Commit message: placing
Parts:
- removed JP4, JP5: Jumper_2_Bridged, symbol Jumper:Jumper_2_Bridged
- added JP10: Jumper_3_Bridged12, Connector_PinHeader_2.54mm:PinHeader_1x03_P2.54mm_Vertical, symbol Jumper:Jumper_3_Bridged12
Connections:
- net 12V0: now also JP10.1 (A)
- net 24V0: now also JP10.3 (B)
- net at A1.8 (VMOT), C16.1, C8.1: now also JP10.2 (C)
Changed lines of the file:
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@@
   (junction (at 97.79 113.03) (diameter 0) (color 0 0 0 0)
   )
-  (junction (at 81.28 44.45) (diameter 0) (color 0 0 0 0)
-  )
   (junction (at 97.79 44.45) (diameter 0) (color 0 0 0 0)
   )
@@
   (junction (at 135.89 44.45) (diameter 0) (color 0 0 0 0)
   )
-  (wire (pts (xy 78.74 44.45) (xy 81.28 44.45))
-    (stroke (width 0) (type default))
-  )
   (wire (pts (xy 97.79 102.87) (xy 97.79 113.03))
     (stroke (width 0) (type default))
@@
     (stroke (width 0) (type default))
   )
-  (wire (pts (xy 78.74 40.64) (xy 81.28 40.64))
-    (stroke (width 0) (type default))
-  )
   (wire (pts (xy 73.66 92.71) (xy 82.55 92.71))
     (stroke (width 0) (type default))
@@
     (stroke (width 0) (type default))
   )
-  (wire (pts (xy 81.28 44.45) (xy 81.28 40.64))
-    (stroke (width 0) (type default))
-  )
   (wire (pts (xy 135.89 53.34) (xy 142.24 53.34))
     (stroke (width 0) (type default))
@@
     (stroke (width 0) (type default))
   )
-  (wire (pts (xy 62.23 44.45) (xy 68.58 44.45))
+  (wire (pts (xy 71.12 50.8) (xy 77.47 50.8))
     (stroke (width 0) (type default))
   )
@@
     (stroke (width 0) (type default))
   )
-  (wire (pts (xy 62.23 40.64) (xy 68.58 40.64))
+  (wire (pts (xy 71.12 38.1) (xy 77.47 38.1))
     (stroke (width 0) (type default))
   )
@@
     (effects (font (size 1.27 1.27)) (justify right))
   )
-  (hierarchical_label "12V0" (shape input) (at 62.23 44.45 180) (fields_autoplaced)
-    (effects (font (size 1.27 1.27)) (justify right))
-  )
-  (hierarchical_label "24V0" (shape input) (at 62.23 40.64 180) (fields_autoplaced)
+  (hierarchical_label "12V0" (shape input) (at 71.12 50.8 180) (fields_autoplaced)
+    (effects (font (size 1.27 1.27)) (justify right))
+  )
+  (hierarchical_label "24V0" (shape input) (at 71.12 38.1 180) (fields_autoplaced)
     (effects (font (size 1.27 1.27)) (justify right))
   )
@@
     )
   )
-  (symbol (lib_id "Jumper:Jumper_2_Bridged") (at 73.66 44.45 0) (unit 1)
-    (in_bom yes) (on_board yes) (dnp no)
-    (property "Reference" "JP5" (at 73.66 45.72 0)
-      (effects (font (size 1.27 1.27)))
-    )
-    (property "Value" "Jumper_2_Bridged" (at 73.66 41.91 0)
-      (effects (font (size 1.27 1.27)) hide)
-    )
-    (property "Footprint" "" (at 73.66 44.45 0)
-      (effects (font (size 1.27 1.27)) hide)
-    )
-    (property "Datasheet" "~" (at 73.66 44.45 0)
+  (symbol (lib_id "Jumper:Jumper_3_Bridged12") (at 77.47 44.45 90) (unit 1)
+    (in_bom yes) (on_board yes) (dnp no) (fields_autoplaced)
+    (property "Reference" "JP10" (at 74.93 43.18 90)
+      (effects (font (size 1.27 1.27)) (justify left))
+    )
+    (property "Value" "Jumper_3_Bridged12" (at 74.93 45.72 90)
+      (effects (font (size 1.27 1.27)) (justify left))
+    )
+    (property "Footprint" "Connector_PinHeader_2.54mm:PinHeader_1x03_P2.54mm_Vertical" (at 77.47 44.45 0)
+      (effects (font (size 1.27 1.27)) hide)
+    )
+    (property "Datasheet" "~" (at 77.47 44.45 0)
       (effects (font (size 1.27 1.27)) hide)
     )
     (pin "1")
     (pin "2")
+    (pin "3")
     (instances
       (project "rollo control"
+        (path "/7fd4875b-e2b3-49e9-a377-320ee6c6aef7/42cd8867-79f6-4c26-8217-42f6d2cc80dc"
+          (reference "JP10") (unit 1)
+        )
+        (path "/7fd4875b-e2b3-49e9-a377-320ee6c6aef7/f84d4e41-04bc-49f0-bae3-d4cb51e0b9a0"
+          (reference "JP7") (unit 1)
+        )
+        (path "/7fd4875b-e2b3-49e9-a377-320ee6c6aef7/4e3087fc-fc79-4dc0-b9f3-dc50efd75935"
+          (reference "JP8") (unit 1)
+        )
         (path "/7fd4875b-e2b3-49e9-a377-320ee6c6aef7/da146848-e1a7-4ab4-bdbb-bdf3e53aad39"
-          (reference "JP5") (unit 1)
+          (reference "JP1") (unit 1)
         )
       )
@@
         )
       )
-    )
-  )
-  (symbol (lib_id "Jumper:Jumper_2_Bridged") (at 73.66 40.64 0) (unit 1)
-    (in_bom yes) (on_board yes) (dnp no)
-    (property "Reference" "JP4" (at 73.66 41.91 0)
-      (effects (font (size 1.27 1.27)))
-    )
-    (property "Value" "Jumper_2_Bridged" (at 73.66 38.1 0)
-      (effects (font (size 1.27 1.27)) hide)
-    )
-    (property "Footprint" "" (at 73.66 40.64 0)
-      (effects (font (size 1.27 1.27)) hide)
-    )
-    (property "Datasheet" "~" (at 73.66 40.64 0)
-      (effects (font (size 1.27 1.27)) hide)
-    )
-    (pin "1")
-    (pin "2")
-    (instances
-      (project "rollo control"
-        (path "/7fd4875b-e2b3-49e9-a377-320ee6c6aef7/da146848-e1a7-4ab4-bdbb-bdf3e53aad39"
-          (reference "JP4") (unit 1)
-        )
-      )
