File: _autosave-rollo control.kicad_pcb (KiCad board)
At the start: 4 copper layers, 100 x 100 mm, 152 parts, among them IC1 IFX007TAUMA1, IC2 IFX007TAUMA1, K1 TIANBO-HJR-4102-L, K2 TIANBO-HJR-4102-L, K3 TIANBO-HJR-4102-L, U1 STM32G071RBTx, U2 AP63205WU, U3 AP7384-33SA, U4 AP7384-50SA, U5 MAX485E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

Commit message: placing
Parts:
- U6: moved to B.Cu
- moved ONE_CON1 118.6 mm to (131.2, 134.9), turned to 0 degrees
- moved ONE_CON2 100.1 mm to (117.8, 134.9), turned to 0 degrees
- moved CON_485_OUT1 98.8 mm to (50.6, 109.1), turned to -90 degrees
- moved CON_485_IN1 97.9 mm to (133.0, 118.9), turned to 90 degrees
- moved FLOW_CON2 81.9 mm to (104.5, 134.9), turned to 0 degrees
- moved FLOW_CON1 64.0 mm to (91.2, 134.9), turned to 0 degrees
- moved R20 56.1 mm to (81.6, 141.1), turned to 90 degrees
- moved R13 52.7 mm to (78.7, 141.1), turned to 90 degrees
- moved R11 49.4 mm to (75.7, 141.1), turned to 90 degrees
- moved BTN_2 46.8 mm to (77.8, 134.9), turned to 0 degrees
- moved R9 46.3 mm to (72.8, 141.1), turned to 90 degrees
- moved D1 45.8 mm to (-5.24, 118.4)
- moved D3 45.8 mm to (-5.24, 121.8)
- moved D4 45.8 mm to (-5.24, 125.1)
- moved R17 45.4 mm to (75.7, 136.4), turned to 90 degrees
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