File: 5V_3V3 DCDC.kicad_sch (KiCad schematic)
At the start: 17 parts, among them U2 AP63205WU, U3 AP7384-33SA, U6 AP7384-50SA

Commit message: ende
Parts:
- removed D10: BAV70S, Package_TO_SOT_SMD:SOT-323_SC-70_Handsoldering, symbol Diode:BAV70S
- added D16: BAV70, Package_TO_SOT_SMD:SOT-23, symbol Diode:BAV70
Connections:
- net 12V0: now also D16.1 (A)
- net 24V0: now also D16.2 (A)
- net at F1.1: now also D16.3 (K)
Other:
- moved on the sheet: F1
Changed lines of the file:
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@@
+    (stroke (width 0) (type default))
+  )
+  (wire (pts (xy 74.93 116.84) (xy 71.12 116.84))
     (stroke (width 0) (type default))
   )
@@
     (stroke (width 0) (type default))
   )
-  (wire (pts (xy 73.66 116.84) (xy 74.93 116.84))
-    (stroke (width 0) (type default))
-  )
   (wire (pts (xy 140.97 82.55) (xy 185.42 82.55))
     (stroke (width 0) (type default))
@@
     (stroke (width 0) (type default))
   )
-  (wire (pts (xy 82.55 121.92) (xy 90.17 121.92))
+  (wire (pts (xy 82.55 121.92) (xy 87.63 121.92))
     (stroke (width 0) (type default))
   )
@@
     (stroke (width 0) (type default))
   )
-  (wire (pts (xy 95.25 121.92) (xy 101.6 121.92))
+  (wire (pts (xy 92.71 121.92) (xy 101.6 121.92))
     (stroke (width 0) (type default))
   )
@@
     (stroke (width 0) (type default))
   )
-  (hierarchical_label "12V0" (shape input) (at 73.66 116.84 180) (fields_autoplaced)
+  (hierarchical_label "12V0" (shape input) (at 71.12 116.84 180) (fields_autoplaced)
     (effects (font (size 1.27 1.27)) (justify right))
   )
@@
     )
   )
-  (symbol (lib_id "Device:Fuse_Small") (at 92.71 121.92 0) (unit 1)
-    (in_bom yes) (on_board yes) (dnp no) (fields_autoplaced)
-    (property "Reference" "F1" (at 92.71 116.84 0)
-      (effects (font (size 1.27 1.27)))
-    )
-    (property "Value" "Fuse_Small" (at 92.71 119.38 0)
-      (effects (font (size 1.27 1.27)))
-    )
-    (property "Footprint" "Fuse:Fuse_1210_3225Metric_Pad1.42x2.65mm_HandSolder" (at 92.71 121.92 0)
-      (effects (font (size 1.27 1.27)) hide)
-    )
-    (property "Datasheet" "~" (at 92.71 121.92 0)
+  (symbol (lib_id "Device:Fuse_Small") (at 90.17 121.92 0) (unit 1)
+    (in_bom yes) (on_board yes) (dnp no) (fields_autoplaced)
+    (property "Reference" "F1" (at 90.17 116.84 0)
+      (effects (font (size 1.27 1.27)))
+    )
+    (property "Value" "Fuse_Small" (at 90.17 119.38 0)
+      (effects (font (size 1.27 1.27)))
+    )
+    (property "Footprint" "Fuse:Fuse_1210_3225Metric_Pad1.42x2.65mm_HandSolder" (at 90.17 121.92 0)
+      (effects (font (size 1.27 1.27)) hide)
+    )
+    (property "Datasheet" "~" (at 90.17 121.92 0)
       (effects (font (size 1.27 1.27)) hide)
     )
@@
         (path "/7fd4875b-e2b3-49e9-a377-320ee6c6aef7/adf5b44f-e84b-4c09-9130-ef2a542c1841"
           (reference "F1") (unit 1)
+        )
+      )
+    )
+  )
+  (symbol (lib_id "Diode:BAV70") (at 82.55 116.84 0) (unit 1)
+    (in_bom yes) (on_board yes) (dnp no) (fields_autoplaced)
+    (property "Reference" "D16" (at 82.55 110.49 0)
+      (effects (font (size 1.27 1.27)))
+    )
+    (property "Value" "BAV70" (at 82.55 113.03 0)
+      (effects (font (size 1.27 1.27)))
+    )
+    (property "Footprint" "Package_TO_SOT_SMD:SOT-23" (at 82.55 116.84 0)
+      (effects (font (size 1.27 1.27)) hide)
+    )
+    (property "Datasheet" "https://assets.nexperia.com/documents/data-sheet/BAV70_SER.pdf" (at 82.55 116.84 0)
+      (effects (font (size 1.27 1.27)) hide)
+    )
+    (pin "1")
+    (pin "2")
+    (pin "3")
+    (instances
+      (project "rollo control"
+        (path "/7fd4875b-e2b3-49e9-a377-320ee6c6aef7/adf5b44f-e84b-4c09-9130-ef2a542c1841"
+          (reference "D16") (unit 1)
         )
       )
@@
         )
       )
-    )
-  )
-  (symbol (lib_id "Diode:BAV70S") (at 82.55 116.84 0) (unit 1)
-    (in_bom yes) (on_board yes) (dnp no) (fields_autoplaced)
-    (property "Reference" "D10" (at 82.55 112.5601 0)
-      (effects (font (size 1.27 1.27)))
-    )
-    (property "Value" "BAV70S" (at 82.55 114.4811 0)
-      (effects (font (size 1.27 1.27)))
-    )
-    (property "Footprint" "Package_TO_SOT_SMD:SOT-323_SC-70_Handsoldering" (at 82.55 116.84 0)
-      (effects (font (size 1.27 1.27)) hide)
-    )
-    (property "Datasheet" "https://assets.nexperia.com/documents/data-sheet/BAV70_SER.pdf" (at 82.55 116.84 0)
-      (effects (font (size 1.27 1.27)) hide)
-    )
-    (pin "1")
-    (pin "2")
-    (pin "6")
-    (pin "3")
-    (pin "4")
-    (pin "5")
-    (instances
-      (project "rollo control"
-        (path "/7fd4875b-e2b3-49e9-a377-320ee6c6aef7/4430fecd-b2bb-44df-a0b9-accae9d9e5ff"
-          (reference "D10") (unit 1)
-        )
-        (path "/7fd4875b-e2b3-49e9-a377-320ee6c6aef7/adf5b44f-e84b-4c09-9130-ef2a542c1841"
-          (reference "D8") (unit 1)
-        )
-      )
