File: 5V_3V3 DCDC.kicad_sch (KiCad schematic)
At the start: 13 parts, among them U3 AP63205WU, U4 AP7384-33SA, U6 AP7384-50SA

Commit message: place
Parts:
- renumbered U3 to U2, U4 to U3
Changed lines of the file:
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@@
     (stroke (width 0) (type default))
   )
-  (wire (pts (xy 204.47 67.31) (xy 214.63 67.31))
+  (wire (pts (xy 204.47 67.31) (xy 223.52 67.31))
     (stroke (width 0) (type default))
   )
@@
     (effects (font (size 1.27 1.27)) (justify right))
   )
-  (hierarchical_label "5V0" (shape input) (at 214.63 67.31 0) (fields_autoplaced)
+  (hierarchical_label "5V0" (shape input) (at 223.52 67.31 0) (fields_autoplaced)
     (effects (font (size 1.27 1.27)) (justify left))
   )
@@
   (symbol (lib_id "Regulator_Linear:AP7384-33SA") (at 191.77 102.87 0) (unit 1)
     (in_bom yes) (on_board yes) (dnp no) (fields_autoplaced)
-    (property "Reference" "U4" (at 191.77 97.9551 0)
+    (property "Reference" "U3" (at 191.77 97.9551 0)
       (effects (font (size 1.27 1.27)))
     )
@@
       (project "rollo control"
         (path "/7fd4875b-e2b3-49e9-a377-320ee6c6aef7/adf5b44f-e84b-4c09-9130-ef2a542c1841"
-          (reference "U4") (unit 1)
+          (reference "U3") (unit 1)
         )
       )
@@
   (symbol (lib_id "Regulator_Switching:AP63205WU") (at 140.97 74.93 0) (unit 1)
     (in_bom yes) (on_board yes) (dnp no) (fields_autoplaced)
-    (property "Reference" "U3" (at 140.97 66.8401 0)
+    (property "Reference" "U2" (at 140.97 66.8401 0)
       (effects (font (size 1.27 1.27)))
     )
@@
       (project "rollo control"
         (path "/7fd4875b-e2b3-49e9-a377-320ee6c6aef7/adf5b44f-e84b-4c09-9130-ef2a542c1841"
-          (reference "U3") (unit 1)
+          (reference "U2") (unit 1)
         )
       )
@@
         )
         (path "/7fd4875b-e2b3-49e9-a377-320ee6c6aef7/adf5b44f-e84b-4c09-9130-ef2a542c1841"
-          (reference "U5") (unit 1)
-        )
-      )
+          (reference "U4") (unit 1)
+        )
+      )

Commit message: 605
Parts:
- added D13, D14: BZV55B5V6, Diode_SMD:D_MiniMELF, symbol Diode:BZV55B5V6
- added D15: BZV55B3V6, Diode_SMD:D_MiniMELF, symbol Diode:BZV55B3V6
- added F1: Fuse_Small, Fuse:Fuse_1210_3225Metric_Pad1.42x2.65mm_HandSolder, symbol Device:Fuse_Small
Connections:
- net 3V3: now also D15.1 (K)
- net 5V0: now also D14.1 (K)
- net 5V0lin: now also D13.1 (K)
- net GND: now also D13.2 (A), D14.2 (A), D15.2 (A)
- net at C21.1, U2.2 (EN), U2.3 (IN)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: now also F1.2; no longer C29.1, D10.6 (K)
- new net: C29.1, D10.6 (K), F1.1
Other:
- moved on the sheet: C22
Changed lines of the file:
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@@
   (junction (at 115.57 82.55) (diameter 0) (color 0 0 0 0)
   )
-  (junction (at 191.77 111.76) (diameter 0) (color 0 0 0 0)
+  (junction (at 134.62 149.86) (diameter 0) (color 0 0 0 0)
   )
   (junction (at 134.62 121.92) (diameter 0) (color 0 0 0 0)
@@
   (junction (at 195.58 67.31) (diameter 0) (color 0 0 0 0)
   )
+  (junction (at 204.47 116.84) (diameter 0) (color 0 0 0 0)
+  )
+  (junction (at 161.29 102.87) (diameter 0) (color 0 0 0 0)
+  )
   (junction (at 105.41 149.86) (diameter 0) (color 0 0 0 0)
   )
@@
   (junction (at 185.42 67.31) (diameter 0) (color 0 0 0 0)
   )
+  (junction (at 214.63 102.87) (diameter 0) (color 0 0 0 0)
+  )
+  (junction (at 191.77 116.84) (diameter 0) (color 0 0 0 0)
+  )
   (junction (at 204.47 67.31) (diameter 0) (color 0 0 0 0)
   )
@@
   (junction (at 115.57 72.39) (diameter 0) (color 0 0 0 0)
   )
+  (junction (at 148.59 149.86) (diameter 0) (color 0 0 0 0)
+  )
   (junction (at 82.55 149.86) (diameter 0) (color 0 0 0 0)
   )
@@
     (stroke (width 0) (type default))
   )
+  (wire (pts (xy 204.47 105.41) (xy 204.47 102.87))
+    (stroke (width 0) (type default))
+  )
   (wire (pts (xy 82.55 129.54) (xy 82.55 149.86))
     (stroke (width 0) (type default))
@@
     (stroke (width 0) (type default))
   )
+  (wire (pts (xy 161.29 102.87) (xy 181.61 102.87))
+    (stroke (width 0) (type default))
+  )
   (wire (pts (xy 134.62 129.54) (xy 134.62 149.86))
     (stroke (width 0) (type default))
   )
+  (wire (pts (xy 214.63 116.84) (xy 204.47 116.84))
+    (stroke (width 0) (type default))
+  )
   (wire (pts (xy 115.57 72.39) (xy 128.27 72.39))
     (stroke (width 0) (type default))
@@
     (stroke (width 0) (type default))
   )
-  (wire (pts (xy 176.53 111.76) (xy 191.77 111.76))
+  (wire (pts (xy 176.53 116.84) (xy 191.77 116.84))
     (stroke (width 0) (type default))
   )
@@
     (stroke (width 0) (type default))
   )
-  (wire (pts (xy 153.67 102.87) (xy 181.61 102.87))
+  (wire (pts (xy 153.67 102.87) (xy 161.29 102.87))
+    (stroke (width 0) (type default))
+  )
+  (wire (pts (xy 191.77 110.49) (xy 191.77 116.84))
     (stroke (width 0) (type default))
   )
@@
     (stroke (width 0) (type default))
   )
-  (wire (pts (xy 204.47 107.95) (xy 204.47 111.76))
+  (wire (pts (xy 204.47 110.49) (xy 204.47 116.84))
     (stroke (width 0) (type default))
   )
@@
     (stroke (width 0) (type default))
   )
+  (wire (pts (xy 161.29 149.86) (xy 148.59 149.86))
+    (stroke (width 0) (type default))
+  )
+  (wire (pts (xy 148.59 137.16) (xy 148.59 149.86))
+    (stroke (width 0) (type default))
+  )
   (wire (pts (xy 154.94 72.39) (xy 154.94 67.31))
     (stroke (width 0) (type default))
@@
     (stroke (width 0) (type default))
   )
+  (wire (pts (xy 214.63 111.76) (xy 214.63 116.84))
+    (stroke (width 0) (type default))
+  )
   (wire (pts (xy 105.41 149.86) (xy 120.65 149.86))
     (stroke (width 0) (type default))
@@
     (stroke (width 0) (type default))
   )
-  (wire (pts (xy 176.53 82.55) (xy 176.53 111.76))
+  (wire (pts (xy 176.53 82.55) (xy 176.53 116.84))
     (stroke (width 0) (type default))
   )
@@
     (stroke (width 0) (type default))
   )
+  (wire (pts (xy 214.63 104.14) (xy 214.63 102.87))
+    (stroke (width 0) (type default))
+  )
   (wire (pts (xy 163.83 74.93) (xy 151.13 74.93))
     (stroke (width 0) (type default))
@@
     (stroke (width 0) (type default))
   )
+  (wire (pts (xy 161.29 115.57) (xy 161.29 149.86))
+    (stroke (width 0) (type default))
+  )
   (wire (pts (xy 134.62 121.92) (xy 134.62 124.46))
     (stroke (width 0) (type default))
   )
-  (wire (pts (xy 191.77 110.49) (xy 191.77 111.76))
-    (stroke (width 0) (type default))
-  )
-  (wire (pts (xy 82.55 121.92) (xy 101.6 121.92))
+  (wire (pts (xy 148.59 149.86) (xy 134.62 149.86))
+    (stroke (width 0) (type default))
+  )
+  (wire (pts (xy 82.55 121.92) (xy 90.17 121.92))
     (stroke (width 0) (type default))
   )
@@
     (stroke (width 0) (type default))
   )
+  (wire (pts (xy 214.63 102.87) (xy 223.52 102.87))
+    (stroke (width 0) (type default))
+  )
   (wire (pts (xy 115.57 78.74) (xy 115.57 82.55))
     (stroke (width 0) (type default))
@@
     (stroke (width 0) (type default))
   )
-  (wire (pts (xy 204.47 111.76) (xy 191.77 111.76))
+  (wire (pts (xy 204.47 116.84) (xy 191.77 116.84))
+    (stroke (width 0) (type default))
+  )
+  (wire (pts (xy 161.29 102.87) (xy 161.29 107.95))
+    (stroke (width 0) (type default))
+  )
+  (wire (pts (xy 95.25 121.92) (xy 101.6 121.92))
     (stroke (width 0) (type default))
   )
@@
   )
   (wire (pts (xy 128.27 77.47) (xy 128.27 72.39))
+    (stroke (width 0) (type default))
+  )
+  (wire (pts (xy 148.59 121.92) (xy 148.59 129.54))
     (stroke (width 0) (type default))
   )
@@
     (effects (font (size 1.27 1.27)) (justify right))
   )
-  (hierarchical_label "3V3" (shape input) (at 214.63 102.87 0) (fields_autoplaced)
+  (hierarchical_label "3V3" (shape input) (at 223.52 102.87 0) (fields_autoplaced)
     (effects (font (size 1.27 1.27)) (justify left))
   )
@@
     )
   )
-  (symbol (lib_id "Device:C_Small") (at 204.47 105.41 0) (unit 1)
+  (symbol (lib_id "Device:Fuse_Small") (at 92.71 121.92 0) (unit 1)
+    (in_bom yes) (on_board yes) (dnp no) (fields_autoplaced)
+    (property "Reference" "F1" (at 92.71 116.84 0)
+      (effects (font (size 1.27 1.27)))
+    )
+    (property "Value" "Fuse_Small" (at 92.71 119.38 0)
+      (effects (font (size 1.27 1.27)))
+    )
+    (property "Footprint" "Fuse:Fuse_1210_3225Metric_Pad1.42x2.65mm_HandSolder" (at 92.71 121.92 0)
+      (effects (font (size 1.27 1.27)) hide)
+    )
+    (property "Datasheet" "~" (at 92.71 121.92 0)
+      (effects (font (size 1.27 1.27)) hide)
+    )
+    (pin "1")
+    (pin "2")
+    (instances
+      (project "rollo control"
+        (path "/7fd4875b-e2b3-49e9-a377-320ee6c6aef7/adf5b44f-e84b-4c09-9130-ef2a542c1841"
+          (reference "F1") (unit 1)
+        )
+      )
+    )
+  )
+  (symbol (lib_id "Diode:BZV55B5V6") (at 148.59 133.35 270) (unit 1)
+    (in_bom yes) (on_board yes) (dnp no) (fields_autoplaced)
+    (property "Reference" "D13" (at 151.13 132.08 90)
+      (effects (font (size 1.27 1.27)) (justify left))
+    )
+    (property "Value" "BZV55B5V6" (at 151.13 134.62 90)
+      (effects (font (size 1.27 1.27)) (justify left))
+    )
+    (property "Footprint" "Diode_SMD:D_MiniMELF" (at 144.145 133.35 0)
+      (effects (font (size 1.27 1.27)) hide)
+    )
+    (property "Datasheet" "https://assets.nexperia.com/documents/data-sheet/BZV55_SER.pdf" (at 148.59 133.35 0)
+      (effects (font (size 1.27 1.27)) hide)
+    )
+    (pin "1")
+    (pin "2")
+    (instances
+      (project "rollo control"
+        (path "/7fd4875b-e2b3-49e9-a377-320ee6c6aef7/adf5b44f-e84b-4c09-9130-ef2a542c1841"
+          (reference "D13") (unit 1)
+        )
+      )
+    )
+  )
+  (symbol (lib_id "Diode:BZV55B3V6") (at 214.63 107.95 270) (unit 1)
+    (in_bom yes) (on_board yes) (dnp no) (fields_autoplaced)
+    (property "Reference" "D15" (at 217.17 106.68 90)
+      (effects (font (size 1.27 1.27)) (justify left))
+    )
+    (property "Value" "BZV55B3V6" (at 217.17 109.22 90)
+      (effects (font (size 1.27 1.27)) (justify left))
+    )
+    (property "Footprint" "Diode_SMD:D_MiniMELF" (at 210.185 107.95 0)
+      (effects (font (size 1.27 1.27)) hide)
+    )
+    (property "Datasheet" "https://assets.nexperia.com/documents/data-sheet/BZV55_SER.pdf" (at 214.63 107.95 0)
+      (effects (font (size 1.27 1.27)) hide)
+    )
+    (pin "1")
+    (pin "2")
+    (instances
+      (project "rollo control"
+        (path "/7fd4875b-e2b3-49e9-a377-320ee6c6aef7/adf5b44f-e84b-4c09-9130-ef2a542c1841"
+          (reference "D15") (unit 1)
+        )
+      )
+    )
+  )
+  (symbol (lib_id "Diode:BZV55B5V6") (at 161.29 111.76 270) (unit 1)
+    (in_bom yes) (on_board yes) (dnp no) (fields_autoplaced)
+    (property "Reference" "D14" (at 163.83 110.49 90)
+      (effects (font (size 1.27 1.27)) (justify left))
+    )
+    (property "Value" "BZV55B5V6" (at 163.83 113.03 90)
+      (effects (font (size 1.27 1.27)) (justify left))
+    )
+    (property "Footprint" "Diode_SMD:D_MiniMELF" (at 156.845 111.76 0)
+      (effects (font (size 1.27 1.27)) hide)
+    )
+    (property "Datasheet" "https://assets.nexperia.com/documents/data-sheet/BZV55_SER.pdf" (at 161.29 111.76 0)
+      (effects (font (size 1.27 1.27)) hide)
+    )
+    (pin "1")
+    (pin "2")
+    (instances
+      (project "rollo control"
+        (path "/7fd4875b-e2b3-49e9-a377-320ee6c6aef7/adf5b44f-e84b-4c09-9130-ef2a542c1841"
+          (reference "D14") (unit 1)
+        )
+      )
+    )
+  )
+  (symbol (lib_id "Device:C_Small") (at 204.47 107.95 0) (unit 1)
     (in_bom yes) (on_board yes) (dnp no)
-    (property "Reference" "C22" (at 206.7941 104.7726 0)
-      (effects (font (size 1.27 1.27)) (justify left))
-    )
-    (property "Value" "10uF" (at 206.7941 106.6936 0)
-      (effects (font (size 1.27 1.27)) (justify left))
-    )
-    (property "Footprint" "" (at 204.47 105.41 0)
-      (effects (font (size 1.27 1.27)) hide)
-    )
-    (property "Datasheet" "~" (at 204.47 105.41 0)
-      (effects (font (size 1.27 1.27)) hide)
-    )
-    (property "Voltage" "50V" (at 208.28 109.22 0)
-      (effects (font (size 1.27 1.27)))
-    )
+    (property "Reference" "C22" (at 206.7941 107.3126 0)
+      (effects (font (size 1.27 1.27)) (justify left))
+    )
+    (property "Value" "10uF" (at 206.7941 109.2336 0)
+      (effects (font (size 1.27 1.27)) (justify left))
+    )
+    (property "Footprint" "" (at 204.47 107.95 0)
+      (effects (font (size 1.27 1.27)) hide)
+    )
+    (property "Datasheet" "~" (at 204.47 107.95 0)
+      (effects (font (size 1.27 1.27)) hide)
+    )
+    (property "Voltage" "50V" (at 208.28 111.76 0)
+      (effects (font (size 1.27 1.27)))
+    )

Commit message: placing
Parts:
- removed C29: C_Small, symbol Device:C_Small
- removed D9: BAV70S, Package_TO_SOT_SMD:SOT-363_SC-70-6, symbol Diode:BAV70S
- added C37: 10uF, Capacitor_SMD:C_1206_3216Metric_Pad1.33x1.80mm_HandSolder, symbol Device:C_Small
- added D10: BAV70S, Package_TO_SOT_SMD:SOT-323_SC-70_Handsoldering, symbol Diode:BAV70S
- C18, C19, C20, C22, C30: footprint (none) -> Capacitor_SMD:C_0805_2012Metric_Pad1.18x1.45mm_HandSolder
- C21: footprint (none) -> Capacitor_SMD:C_1206_3216Metric_Pad1.33x1.80mm_HandSolder
- D10: footprint Package_TO_SOT_SMD:SOT-363_SC-70-6 -> Package_TO_SOT_SMD:SOT-323_SC-70_Handsoldering
Connections:
- net 5V0: now also D10.6 (K)
- net 5V0lin: now also D10.1 (A)
- net GND: now also C37.2
- net at C21.1, F1.2, U2.2 (EN)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: now also C37.1

Commit message: gsdfg
dyfg
Parts:
- removed D10: BAV70S, Package_TO_SOT_SMD:SOT-323_SC-70_Handsoldering, symbol Diode:BAV70S
- removed F1: Fuse_Small, Fuse:Fuse_1210_3225Metric_Pad1.42x2.65mm_HandSolder, symbol Device:Fuse_Small
- removed U6: AP7384-50SA, Package_TO_SOT_SMD:SOT-23, symbol Regulator_Linear:AP7384-50SA
- added U9: L7805, Package_TO_SOT_SMD:SOT-223, symbol Regulator_Linear:L7805
Connections:
- net 12V0: now also C21.1, C37.1, U2.2 (EN), U2.3 (IN), U9.1 (IN)
- net 5V0lin: now also U9.3 (OUT)
- net GND: now also U9.2 (GND)
Changed lines of the file:
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@@
-    (stroke (width 0) (type default))
-  )
-  (wire (pts (xy 90.17 110.49) (xy 90.17 116.84))
     (stroke (width 0) (type default))
   )
@@
     (stroke (width 0) (type default))
   )
-  (wire (pts (xy 73.66 116.84) (xy 74.93 116.84))
-    (stroke (width 0) (type default))
-  )
   (wire (pts (xy 140.97 82.55) (xy 185.42 82.55))
     (stroke (width 0) (type default))
   )
-  (wire (pts (xy 73.66 110.49) (xy 90.17 110.49))
-    (stroke (width 0) (type default))
-  )
   (wire (pts (xy 101.6 134.62) (xy 101.6 149.86))
     (stroke (width 0) (type default))
   )
+  (wire (pts (xy 82.55 121.92) (xy 101.6 121.92))
+    (stroke (width 0) (type default))
+  )
   (wire (pts (xy 185.42 67.31) (xy 195.58 67.31))
     (stroke (width 0) (type default))
@@
     (stroke (width 0) (type default))
   )
-  (wire (pts (xy 82.55 121.92) (xy 90.17 121.92))
-    (stroke (width 0) (type default))
-  )
   (wire (pts (xy 115.57 82.55) (xy 140.97 82.55))
     (stroke (width 0) (type default))
@@
     (stroke (width 0) (type default))
   )
-  (wire (pts (xy 95.25 121.92) (xy 101.6 121.92))
-    (stroke (width 0) (type default))
-  )
   (wire (pts (xy 199.39 102.87) (xy 204.47 102.87))
     (stroke (width 0) (type default))
@@
     (stroke (width 0) (type default))
   )
-  (hierarchical_label "12V0" (shape input) (at 73.66 116.84 180) (fields_autoplaced)
-    (effects (font (size 1.27 1.27)) (justify right))
-  )
-  (hierarchical_label "24V0" (shape input) (at 73.66 110.49 180) (fields_autoplaced)
+  (hierarchical_label "12V0" (shape input) (at 82.55 121.92 180) (fields_autoplaced)
     (effects (font (size 1.27 1.27)) (justify right))
   )
@@
     (effects (font (size 1.27 1.27)) (justify right))
   )
+  (symbol (lib_id "Regulator_Linear:L7805") (at 120.65 121.92 0) (unit 1)
+    (in_bom yes) (on_board yes) (dnp no) (fields_autoplaced)
+    (property "Reference" "U9" (at 120.65 115.57 0)
+      (effects (font (size 1.27 1.27)))
+    )
+    (property "Value" "L7805" (at 120.65 118.11 0)
+      (effects (font (size 1.27 1.27)))
+    )
+    (property "Footprint" "Package_TO_SOT_SMD:SOT-223" (at 121.285 125.73 0)
+      (effects (font (size 1.27 1.27) italic) (justify left) hide)
+    )
+    (property "Datasheet" "http://www.st.com/content/ccc/resource/technical/document/datasheet/41/4f/b3/b0/12/d4/47/88/CD00000444.pdf/files/CD00000444.pdf/jcr:content/translations/en.CD00000444.pdf" (at 120.65 123.19 0)
+      (effects (font (size 1.27 1.27)) hide)
+    )
+    (pin "1")
+    (pin "2")
+    (pin "3")
+    (instances
+      (project "rollo control"
+        (path "/7fd4875b-e2b3-49e9-a377-320ee6c6aef7/adf5b44f-e84b-4c09-9130-ef2a542c1841"
+          (reference "U9") (unit 1)
+        )
+      )
+    )
+  )
   (symbol (lib_id "Device:C_Small") (at 163.83 71.12 0) (unit 1)
     (in_bom yes) (on_board yes) (dnp no)
@@
         (path "/7fd4875b-e2b3-49e9-a377-320ee6c6aef7/adf5b44f-e84b-4c09-9130-ef2a542c1841"
           (reference "C24") (unit 1)
-        )
-      )
-    )
-  )
-  (symbol (lib_id "Device:Fuse_Small") (at 92.71 121.92 0) (unit 1)
-    (in_bom yes) (on_board yes) (dnp no) (fields_autoplaced)
-    (property "Reference" "F1" (at 92.71 116.84 0)
-      (effects (font (size 1.27 1.27)))
-    )
-    (property "Value" "Fuse_Small" (at 92.71 119.38 0)
-      (effects (font (size 1.27 1.27)))
-    )
-    (property "Footprint" "Fuse:Fuse_1210_3225Metric_Pad1.42x2.65mm_HandSolder" (at 92.71 121.92 0)
-      (effects (font (size 1.27 1.27)) hide)
-    )
-    (property "Datasheet" "~" (at 92.71 121.92 0)
-      (effects (font (size 1.27 1.27)) hide)
-    )
-    (pin "1")
-    (pin "2")
-    (instances
-      (project "rollo control"
-        (path "/7fd4875b-e2b3-49e9-a377-320ee6c6aef7/adf5b44f-e84b-4c09-9130-ef2a542c1841"
-          (reference "F1") (unit 1)
         )
       )
@@
         )
       )
-    )
-  )
-  (symbol (lib_id "Diode:BAV70S") (at 82.55 116.84 0) (unit 1)
-    (in_bom yes) (on_board yes) (dnp no) (fields_autoplaced)
-    (property "Reference" "D10" (at 82.55 112.5601 0)
-      (effects (font (size 1.27 1.27)))
-    )
-    (property "Value" "BAV70S" (at 82.55 114.4811 0)
-      (effects (font (size 1.27 1.27)))
-    )
-    (property "Footprint" "Package_TO_SOT_SMD:SOT-323_SC-70_Handsoldering" (at 82.55 116.84 0)
-      (effects (font (size 1.27 1.27)) hide)
-    )
-    (property "Datasheet" "https://assets.nexperia.com/documents/data-sheet/BAV70_SER.pdf" (at 82.55 116.84 0)
-      (effects (font (size 1.27 1.27)) hide)
-    )
-    (pin "1")
-    (pin "2")
-    (pin "6")
-    (pin "3")
-    (pin "4")
-    (pin "5")
-    (instances
-      (project "rollo control"
-        (path "/7fd4875b-e2b3-49e9-a377-320ee6c6aef7/4430fecd-b2bb-44df-a0b9-accae9d9e5ff"
-          (reference "D10") (unit 1)
-        )
-        (path "/7fd4875b-e2b3-49e9-a377-320ee6c6aef7/adf5b44f-e84b-4c09-9130-ef2a542c1841"
-          (reference "D8") (unit 1)
-        )
-      )
-    )
-  )
-  (symbol (lib_id "Regulator_Linear:AP7384-50SA") (at 120.65 121.92 0) (unit 1)
-    (in_bom yes) (on_board yes) (dnp no) (fields_autoplaced)
-    (property "Reference" "U6" (at 120.65 117.0051 0)
-      (effects (font (size 1.27 1.27)))
-    )
-    (property "Value" "AP7384-50SA" (at 120.65 118.9261 0)
-      (effects (font (size 1.27 1.27)))
-    )
-    (property "Footprint" "Package_TO_SOT_SMD:SOT-23" (at 120.65 116.205 0)
-      (effects (font (size 1.27 1.27) italic) hide)
-    )
-    (property "Datasheet" "https://www.diodes.com/assets/Datasheets/AP7384.pdf" (at 120.65 123.19 0)
-      (effects (font (size 1.27 1.27)) hide)
-    )
-    (pin "1")
-    (pin "2")
-    (pin "3")
-    (instances
-      (project "rollo control"
-        (path "/7fd4875b-e2b3-49e9-a377-320ee6c6aef7/4430fecd-b2bb-44df-a0b9-accae9d9e5ff"
-          (reference "U6") (unit 1)
-        )
-        (path "/7fd4875b-e2b3-49e9-a377-320ee6c6aef7/adf5b44f-e84b-4c09-9130-ef2a542c1841"
-          (reference "U4") (unit 1)
-        )
-      )
