File: Analog24-12.kicad_sch (KiCad schematic)
At the start: 24 parts

Commit message: gsdfg
dyfg
Parts:
- removed C30: C_Small, Capacitor_SMD:C_0603_1608Metric_Pad1.08x0.95mm_HandSolder, symbol Device:C_Small
- removed D1 (x2): SP0502BAHT, Package_TO_SOT_SMD:SOT-23, symbol Power_Protection:SP0502BAHT
- removed R34, R35: ~, Resistor_SMD:R_0201_0603Metric_Pad0.64x0.40mm_HandSolder, symbol Device:R_Small
Connections:
- net 24V_SIG is gone; now on net 12V_SIG: C29.1, R33.1, R36.2
