File: RS485niso.kicad_sch (KiCad schematic)
At the start: 9 parts, among them J4 Conn_01x02, U6 MAX485E

Commit message: place
Parts:
- removed J4: Conn_01x02, Connector_Phoenix_MSTB:PhoenixContact_MSTBA_2,5_2-G-5,08_1x02_P5.08mm_Horizontal, symbol Connector_Generic:Conn_01x02
- added CON_485_IN1, CON_485_OUT1: Conn_01x04, Connector_Phoenix_MC:PhoenixContact_MC_1,5_4-G-3.81_1x04_P3.81mm_Horizontal, symbol Connector_Generic:Conn_01x04
- renumbered U6 to U5
Connections:
- net 5V0: now also CON_485_IN1.1 (Pin_1), CON_485_OUT1.1 (Pin_1)
- net GND: now also CON_485_IN1.4 (Pin_4), CON_485_OUT1.4 (Pin_4)
- net at D9.1 (K), R26.1, R27.2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: now also CON_485_IN1.3 (Pin_3), CON_485_OUT1.3 (Pin_3)
- net at D9.2 (K), R24.1, R25.2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: now also CON_485_IN1.2 (Pin_2), CON_485_OUT1.2 (Pin_2)
Changed lines of the file:
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@@
   (junction (at 162.56 78.74) (diameter 0) (color 0 0 0 0)
   )
+  (junction (at 200.66 81.28) (diameter 0) (color 0 0 0 0)
+  )
   (junction (at 162.56 101.6) (diameter 0) (color 0 0 0 0)
   )
@@
   (junction (at 114.3 81.28) (diameter 0) (color 0 0 0 0)
   )
+  (junction (at 198.12 83.82) (diameter 0) (color 0 0 0 0)
+  )
   (wire (pts (xy 162.56 96.52) (xy 162.56 101.6))
     (stroke (width 0) (type default))
@@
     (stroke (width 0) (type default))
   )
-  (wire (pts (xy 186.69 85.09) (xy 186.69 86.36))
+  (wire (pts (xy 186.69 83.82) (xy 186.69 86.36))
     (stroke (width 0) (type default))
   )
@@
     (stroke (width 0) (type default))
   )
+  (wire (pts (xy 195.58 99.06) (xy 203.2 99.06))
+    (stroke (width 0) (type default))
+  )
+  (wire (pts (xy 198.12 83.82) (xy 186.69 83.82))
+    (stroke (width 0) (type default))
+  )
   (wire (pts (xy 129.54 52.07) (xy 129.54 57.15))
     (stroke (width 0) (type default))
@@
     (stroke (width 0) (type default))
   )
-  (wire (pts (xy 193.04 82.55) (xy 186.69 82.55))
+  (wire (pts (xy 203.2 81.28) (xy 200.66 81.28))
     (stroke (width 0) (type default))
   )
@@
     (stroke (width 0) (type default))
   )
+  (wire (pts (xy 200.66 81.28) (xy 186.69 81.28))
+    (stroke (width 0) (type default))
+  )
   (wire (pts (xy 172.72 86.36) (xy 172.72 88.9))
     (stroke (width 0) (type default))
   )
+  (wire (pts (xy 195.58 78.74) (xy 203.2 78.74))
+    (stroke (width 0) (type default))
+  )
   (wire (pts (xy 177.8 78.74) (xy 186.69 78.74))
     (stroke (width 0) (type default))
   )
-  (wire (pts (xy 193.04 85.09) (xy 186.69 85.09))
+  (wire (pts (xy 195.58 91.44) (xy 203.2 91.44))
+    (stroke (width 0) (type default))
+  )
+  (wire (pts (xy 203.2 83.82) (xy 198.12 83.82))
     (stroke (width 0) (type default))
   )
@@
     (stroke (width 0) (type default))
   )
+  (wire (pts (xy 203.2 96.52) (xy 198.12 96.52))
+    (stroke (width 0) (type default))
+  )
   (wire (pts (xy 162.56 86.36) (xy 162.56 88.9))
     (stroke (width 0) (type default))
@@
     (stroke (width 0) (type default))
   )
-  (wire (pts (xy 186.69 82.55) (xy 186.69 78.74))
+  (wire (pts (xy 186.69 81.28) (xy 186.69 78.74))
     (stroke (width 0) (type default))
   )
@@
     (stroke (width 0) (type default))
   )
+  (wire (pts (xy 203.2 93.98) (xy 200.66 93.98))
+    (stroke (width 0) (type default))
+  )
+  (wire (pts (xy 198.12 96.52) (xy 198.12 83.82))
+    (stroke (width 0) (type default))
+  )
   (wire (pts (xy 175.26 101.6) (xy 162.56 101.6))
     (stroke (width 0) (type default))
   )
+  (wire (pts (xy 200.66 93.98) (xy 200.66 81.28))
+    (stroke (width 0) (type default))
+  )
   (wire (pts (xy 129.54 101.6) (xy 129.54 105.41))
     (stroke (width 0) (type default))
@@
   )
   (wire (pts (xy 139.7 86.36) (xy 147.32 86.36))
+    (stroke (width 0) (type default))
+  )
+  (wire (pts (xy 195.58 86.36) (xy 203.2 86.36))
     (stroke (width 0) (type default))
   )
@@
     (effects (font (size 1.27 1.27)) (justify right))
   )
+  (hierarchical_label "5V0" (shape input) (at 195.58 78.74 180) (fields_autoplaced)
+    (effects (font (size 1.27 1.27)) (justify right))
+  )
+  (hierarchical_label "5V0" (shape input) (at 195.58 91.44 180) (fields_autoplaced)
+    (effects (font (size 1.27 1.27)) (justify right))
+  )
+  (hierarchical_label "GND" (shape input) (at 195.58 99.06 180) (fields_autoplaced)
+    (effects (font (size 1.27 1.27)) (justify right))
+  )
   (hierarchical_label "485_poci" (shape input) (at 110.49 78.74 180) (fields_autoplaced)
+    (effects (font (size 1.27 1.27)) (justify right))
+  )
+  (hierarchical_label "GND" (shape input) (at 195.58 86.36 180) (fields_autoplaced)
     (effects (font (size 1.27 1.27)) (justify right))
   )
@@
   (hierarchical_label "485_enable" (shape input) (at 110.49 81.28 180) (fields_autoplaced)
     (effects (font (size 1.27 1.27)) (justify right))
+  )
+  (symbol (lib_id "Connector_Generic:Conn_01x04") (at 208.28 81.28 0) (unit 1)
+    (in_bom yes) (on_board yes) (dnp no) (fields_autoplaced)
+    (property "Reference" "CON_485_IN1" (at 210.312 81.9063 0)
+      (effects (font (size 1.27 1.27)) (justify left))
+    )
+    (property "Value" "Conn_01x04" (at 210.312 83.8273 0)
+      (effects (font (size 1.27 1.27)) (justify left))
+    )
+    (property "Footprint" "Connector_Phoenix_MC:PhoenixContact_MC_1,5_4-G-3.81_1x04_P3.81mm_Horizontal" (at 208.28 81.28 0)
+      (effects (font (size 1.27 1.27)) hide)
+    )
+    (property "Datasheet" "~" (at 208.28 81.28 0)
+      (effects (font (size 1.27 1.27)) hide)
+    )
+    (pin "1")
+    (pin "2")
+    (pin "3")
+    (pin "4")
+    (instances
+      (project "rollo control"
+        (path "/7fd4875b-e2b3-49e9-a377-320ee6c6aef7/b6c73591-e73a-4bd7-89c6-628af8fa635f"
+          (reference "CON_485_IN1") (unit 1)
+        )
+      )
+    )
   )
   (symbol (lib_id "Device:R") (at 162.56 92.71 180) (unit 1)
@@
     )
   )
-  (symbol (lib_id "Connector_Generic:Conn_01x02") (at 198.12 82.55 0) (unit 1)
-    (in_bom yes) (on_board yes) (dnp no) (fields_autoplaced)
-    (property "Reference" "J4" (at 200.152 83.1763 0)
-      (effects (font (size 1.27 1.27)) (justify left))
-    )
-    (property "Value" "Conn_01x02" (at 200.152 85.0973 0)
-      (effects (font (size 1.27 1.27)) (justify left))
-    )
-    (property "Footprint" "Connector_Phoenix_MSTB:PhoenixContact_MSTBA_2,5_2-G-5,08_1x02_P5.08mm_Horizontal" (at 198.12 82.55 0)
-      (effects (font (size 1.27 1.27)) hide)
-    )
-    (property "Datasheet" "~" (at 198.12 82.55 0)
-      (effects (font (size 1.27 1.27)) hide)
-    )
-    (pin "1")
-    (pin "2")
-    (instances
-      (project "rollo control"
-        (path "/7fd4875b-e2b3-49e9-a377-320ee6c6aef7/f84d4e41-04bc-49f0-bae3-d4cb51e0b9a0"
-          (reference "J4") (unit 1)
-        )
-        (path "/7fd4875b-e2b3-49e9-a377-320ee6c6aef7/b6c73591-e73a-4bd7-89c6-628af8fa635f"
-          (reference "CON_1") (unit 1)
-        )
-      )
-    )
-  )
   (symbol (lib_id "Interface_UART:MAX485E") (at 129.54 81.28 0) (unit 1)
     (in_bom yes) (on_board yes) (dnp no) (fields_autoplaced)
-    (property "Reference" "U6" (at 131.4959 68.1101 0)
+    (property "Reference" "U5" (at 131.4959 68.1101 0)
       (effects (font (size 1.27 1.27)) (justify left))
     )
@@
       (project "rollo control"
         (path "/7fd4875b-e2b3-49e9-a377-320ee6c6aef7/b6c73591-e73a-4bd7-89c6-628af8fa635f"
-          (reference "U6") (unit 1)
+          (reference "U5") (unit 1)
         )
       )
@@
   )
   (symbol (lib_id "Power_Protection:SP0502BAHT") (at 175.26 93.98 0) (unit 1)
-    (in_bom yes) (on_board yes) (dnp no) (fields_autoplaced)
-    (property "Reference" "D9" (at 180.467 93.3363 0)
-      (effects (font (size 1.27 1.27)) (justify left))
-    )
-    (property "Value" "SP0502BAHT" (at 180.467 95.2573 0)
+    (in_bom yes) (on_board yes) (dnp no)
+    (property "Reference" "D9" (at 170.18 104.14 0)
+      (effects (font (size 1.27 1.27)) (justify left))
+    )
+    (property "Value" "SP0502BAHT" (at 170.18 106.68 0)
       (effects (font (size 1.27 1.27)) (justify left))
     )
@@
         )
       )
+    )
+  )
+  (symbol (lib_id "Connector_Generic:Conn_01x04") (at 208.28 93.98 0) (unit 1)
+    (in_bom yes) (on_board yes) (dnp no) (fields_autoplaced)
+    (property "Reference" "CON_485_OUT1" (at 210.312 94.6063 0)
+      (effects (font (size 1.27 1.27)) (justify left))
+    )
+    (property "Value" "Conn_01x04" (at 210.312 96.5273 0)
+      (effects (font (size 1.27 1.27)) (justify left))
+    )
+    (property "Footprint" "Connector_Phoenix_MC:PhoenixContact_MC_1,5_4-G-3.81_1x04_P3.81mm_Horizontal" (at 208.28 93.98 0)
+      (effects (font (size 1.27 1.27)) hide)
+    )
+    (property "Datasheet" "~" (at 208.28 93.98 0)
+      (effects (font (size 1.27 1.27)) hide)
+    )
+    (pin "1")
+    (pin "2")
+    (pin "3")
+    (pin "4")
+    (instances
+      (project "rollo control"
+        (path "/7fd4875b-e2b3-49e9-a377-320ee6c6aef7/b6c73591-e73a-4bd7-89c6-628af8fa635f"
+          (reference "CON_485_OUT1") (unit 1)
+        )
+      )

Commit message: mc1.5
Parts:
- CON_485_IN1, CON_485_OUT1: footprint Connector_Phoenix_MC:PhoenixContact_MC_1,5_4-G-3.81_1x04_P3.81mm_Horizontal -> Connector_Phoenix_MC:PhoenixContact_MC_1,5_4-G-3.5_1x04_P3.50mm_Horizontal
Changed lines of the file:
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@@
       (effects (font (size 1.27 1.27)) (justify left))
     )
-    (property "Footprint" "Connector_Phoenix_MC:PhoenixContact_MC_1,5_4-G-3.81_1x04_P3.81mm_Horizontal" (at 208.28 81.28 0)
+    (property "Footprint" "Connector_Phoenix_MC:PhoenixContact_MC_1,5_4-G-3.5_1x04_P3.50mm_Horizontal" (at 208.28 81.28 0)
       (effects (font (size 1.27 1.27)) hide)
     )
-    (property "Datasheet" "~" (at 208.28 81.28 0)
+    (property "Datasheet" "" (at 208.28 81.28 0)
       (effects (font (size 1.27 1.27)) hide)
     )
@@
       (effects (font (size 1.27 1.27)) (justify left))
     )
-    (property "Footprint" "Connector_Phoenix_MC:PhoenixContact_MC_1,5_4-G-3.81_1x04_P3.81mm_Horizontal" (at 208.28 93.98 0)
+    (property "Footprint" "Connector_Phoenix_MC:PhoenixContact_MC_1,5_4-G-3.5_1x04_P3.50mm_Horizontal" (at 208.28 93.98 0)
       (effects (font (size 1.27 1.27)) hide)
     )

Commit message: 605
Parts:
- R24, R25, R26, R27, R28: footprint Resistor_SMD:R_0805_2012Metric_Pad1.20x1.40mm_HandSolder -> Resistor_SMD:R_0201_0603Metric_Pad0.64x0.40mm_HandSolder
Changed lines of the file:
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@@
       (effects (font (size 1.27 1.27)) (justify right))
     )
-    (property "Footprint" "Resistor_SMD:R_0805_2012Metric_Pad1.20x1.40mm_HandSolder" (at 164.338 92.71 90)
+    (property "Footprint" "Resistor_SMD:R_0201_0603Metric_Pad0.64x0.40mm_HandSolder" (at 164.338 92.71 90)
       (effects (font (size 1.27 1.27)) hide)
     )
@@
       (effects (font (size 1.27 1.27)) (justify right))
     )
-    (property "Footprint" "Resistor_SMD:R_0805_2012Metric_Pad1.20x1.40mm_HandSolder" (at 164.338 72.39 90)
+    (property "Footprint" "Resistor_SMD:R_0201_0603Metric_Pad0.64x0.40mm_HandSolder" (at 164.338 72.39 90)
       (effects (font (size 1.27 1.27)) hide)
     )
@@
       (effects (font (size 1.27 1.27)))
     )
-    (property "Footprint" "Resistor_SMD:R_0805_2012Metric_Pad1.20x1.40mm_HandSolder" (at 151.13 88.138 90)
+    (property "Footprint" "Resistor_SMD:R_0201_0603Metric_Pad0.64x0.40mm_HandSolder" (at 151.13 88.138 90)
       (effects (font (size 1.27 1.27)) hide)
     )
@@
       (effects (font (size 1.27 1.27)))
     )
-    (property "Footprint" "Resistor_SMD:R_0805_2012Metric_Pad1.20x1.40mm_HandSolder" (at 151.13 80.518 90)
+    (property "Footprint" "Resistor_SMD:R_0201_0603Metric_Pad0.64x0.40mm_HandSolder" (at 151.13 80.518 90)
       (effects (font (size 1.27 1.27)) hide)
     )
@@
       (effects (font (size 1.27 1.27)) (justify right))
     )
-    (property "Footprint" "Resistor_SMD:R_0805_2012Metric_Pad1.20x1.40mm_HandSolder" (at 164.338 82.55 90)
-      (effects (font (size 1.27 1.27)) hide)
-    )
+    (property "Footprint" "Resistor_SMD:R_0201_0603Metric_Pad0.64x0.40mm_HandSolder" (at 164.338 82.55 90)
+      (effects (font (size 1.27 1.27)) hide)
+    )

Commit message: ende
Parts:
- R24, R25, R26, R27, R28: footprint Resistor_SMD:R_0201_0603Metric_Pad0.64x0.40mm_HandSolder -> Resistor_SMD:R_0805_2012Metric_Pad1.20x1.40mm_HandSolder
Changed lines of the file:
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@@
       (effects (font (size 1.27 1.27)) (justify right))
     )
-    (property "Footprint" "Resistor_SMD:R_0201_0603Metric_Pad0.64x0.40mm_HandSolder" (at 164.338 92.71 90)
+    (property "Footprint" "Resistor_SMD:R_0805_2012Metric_Pad1.20x1.40mm_HandSolder" (at 164.338 92.71 90)
       (effects (font (size 1.27 1.27)) hide)
     )
@@
       (effects (font (size 1.27 1.27)) (justify right))
     )
-    (property "Footprint" "Resistor_SMD:R_0201_0603Metric_Pad0.64x0.40mm_HandSolder" (at 164.338 72.39 90)
+    (property "Footprint" "Resistor_SMD:R_0805_2012Metric_Pad1.20x1.40mm_HandSolder" (at 164.338 72.39 90)
       (effects (font (size 1.27 1.27)) hide)
     )
@@
       (effects (font (size 1.27 1.27)))
     )
-    (property "Footprint" "Resistor_SMD:R_0201_0603Metric_Pad0.64x0.40mm_HandSolder" (at 151.13 88.138 90)
+    (property "Footprint" "Resistor_SMD:R_0805_2012Metric_Pad1.20x1.40mm_HandSolder" (at 151.13 88.138 90)
       (effects (font (size 1.27 1.27)) hide)
     )
@@
       (effects (font (size 1.27 1.27)))
     )
-    (property "Footprint" "Resistor_SMD:R_0201_0603Metric_Pad0.64x0.40mm_HandSolder" (at 151.13 80.518 90)
+    (property "Footprint" "Resistor_SMD:R_0805_2012Metric_Pad1.20x1.40mm_HandSolder" (at 151.13 80.518 90)
       (effects (font (size 1.27 1.27)) hide)
     )
@@
       (effects (font (size 1.27 1.27)) (justify right))
     )
-    (property "Footprint" "Resistor_SMD:R_0201_0603Metric_Pad0.64x0.40mm_HandSolder" (at 164.338 82.55 90)
-      (effects (font (size 1.27 1.27)) hide)
-    )
+    (property "Footprint" "Resistor_SMD:R_0805_2012Metric_Pad1.20x1.40mm_HandSolder" (at 164.338 82.55 90)
+      (effects (font (size 1.27 1.27)) hide)
+    )
