File: rollo control.kicad_sch (KiCad schematic)
At the start: 6 parts

Commit message: ende
Connections:
- net 12V0 renamed Analog-IN/12V0
- net 24V0 renamed Analog-IN/24V0
Other:
- sheet mcu-relais ports: added none; removed 24V0
Changed lines of the file:
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@@
 (kicad_sch (version 20230121) (generator eeschema)
   (paper "A4")
+  (bus_alias "Din" (members "I2C_SDA" "I2C_SCL" "FLW_Sig1" "FLW_Sig2" "BTN_1" "BTN_2" "ONE_SIG" ""))
+  (bus_alias "485" (members "poci" "pico" "enable" ""))
+  (bus_alias "Autoterm" (members "RX" "TX"))
+  (bus_alias "DCDrive" (members "IFX1_FB" "IFX1_IN" "IFX1_INH" "IFX2_FB" "IFX2_IN" "IFX2_INH"))
+  (bus_alias "Stepper" (members "Step_step" "Step_dir" "Step_MS1" "Step_MS2" "Step_MS3" "Step_enable" "Step_sleep" "Step_reset"))
   (bus_alias "Ain" (members "Ain_ntc0+" "Ain_ntc0-" "Ain_12V_Sig" "Ain_24V_Sig" "Ain_ntc1+" "Ain_ntc1-"))
+  (bus_alias "Rel" (members "REL1" "REL2" "REL3" "REL4" "REL5" "REL6" "REL7"))
   (bus_alias "SolidState" (members "pump1" "pump2" "pump3" "pump4" "pump_fb2" "pump_fb1"))
-  (bus_alias "Rel" (members "REL1" "REL2" "REL3" "REL4" "REL5" "REL6" "REL7"))
-  (bus_alias "DCDrive" (members "IFX1_FB" "IFX1_IN" "IFX1_INH" "IFX2_FB" "IFX2_IN" "IFX2_INH"))
-  (bus_alias "Autoterm" (members "RX" "TX"))
-  (bus_alias "Din" (members "I2C_SDA" "I2C_SCL" "FLW_Sig1" "FLW_Sig2" "BTN_1" "BTN_2" "ONE_SIG" ""))
-  (bus_alias "Stepper" (members "Step_step" "Step_dir" "Step_MS1" "Step_MS2" "Step_MS3" "Step_enable" "Step_sleep" "Step_reset"))
-  (bus_alias "485" (members "poci" "pico" "enable" ""))
   (junction (at 124.46 82.55) (diameter 0) (color 0 0 0 0)
   )
-  (junction (at 49.53 43.18) (diameter 0) (color 0 0 0 0)
-  )
   (junction (at 146.05 43.18) (diameter 0) (color 0 0 0 0)
   )
@@
   (junction (at 82.55 82.55) (diameter 0) (color 0 0 0 0)
   )
+  (junction (at 35.56 58.42) (diameter 0) (color 0 0 0 0)
+  )
   (junction (at 149.86 88.9) (diameter 0) (color 0 0 0 0)
   )
@@
   (junction (at 143.51 85.09) (diameter 0) (color 0 0 0 0)
   )
-  (junction (at 54.61 46.99) (diameter 0) (color 0 0 0 0)
-  )
   (junction (at 30.48 74.93) (diameter 0) (color 0 0 0 0)
   )
-  (junction (at 35.56 68.58) (diameter 0) (color 0 0 0 0)
+  (junction (at 33.02 68.58) (diameter 0) (color 0 0 0 0)
   )
   (junction (at 63.5 85.09) (diameter 0) (color 0 0 0 0)
@@
   (junction (at 76.2 60.96) (diameter 0) (color 0 0 0 0)
   )
-  (junction (at 33.02 58.42) (diameter 0) (color 0 0 0 0)
-  )
   (bus_entry (at 124.46 114.3) (size 2.54 -2.54)
     (stroke (width 0) (type default))
@@
     (stroke (width 0) (type default))
   )
+  (wire (pts (xy 33.02 68.58) (xy 33.02 90.17))
+    (stroke (width 0) (type default))
+  )
   (wire (pts (xy 157.48 62.23) (xy 168.91 62.23))
     (stroke (width 0) (type default))
@@
     (stroke (width 0) (type default))
   )
-  (wire (pts (xy 218.44 101.6) (xy 218.44 106.68))
-    (stroke (width 0) (type default))
-  )
   (bus (pts (xy 154.94 72.39) (xy 154.94 74.93))
     (stroke (width 0) (type default))
@@
     (stroke (width 0) (type default))
   )
+  (wire (pts (xy 33.02 64.77) (xy 39.37 64.77))
+    (stroke (width 0) (type default))
+  )
   (bus (pts (xy 160.02 124.46) (xy 160.02 127))
     (stroke (width 0) (type default))
@@
     (stroke (width 0) (type default))
   )
-  (wire (pts (xy 35.56 90.17) (xy 35.56 68.58))
-    (stroke (width 0) (type default))
-  )
   (wire (pts (xy 181.61 85.09) (xy 203.2 85.09))
     (stroke (width 0) (type default))
@@
     (stroke (width 0) (type default))
   )
-  (wire (pts (xy 33.02 80.01) (xy 33.02 58.42))
-    (stroke (width 0) (type default))
-  )
   (bus (pts (xy 72.39 114.3) (xy 72.39 116.84))
     (stroke (width 0) (type default))
@@
     (stroke (width 0) (type default))
   )
-  (wire (pts (xy 33.02 58.42) (xy 39.37 58.42))
-    (stroke (width 0) (type default))
-  )
   (wire (pts (xy 215.9 132.08) (xy 246.38 132.08))
     (stroke (width 0) (type default))
@@
     (stroke (width 0) (type default))
   )
-  (wire (pts (xy 27.94 68.58) (xy 35.56 68.58))
-    (stroke (width 0) (type default))
-  )
   (bus (pts (xy 160.02 82.55) (xy 187.96 82.55))
     (stroke (width 0) (type default))
@@
     (stroke (width 0) (type default))
   )
+  (wire (pts (xy 35.56 80.01) (xy 35.56 58.42))
+    (stroke (width 0) (type default))
+  )
   (wire (pts (xy 157.48 69.85) (xy 168.91 69.85))
     (stroke (width 0) (type default))
@@
     (stroke (width 0) (type default))
   )
+  (wire (pts (xy 99.06 101.6) (xy 49.53 101.6))
+    (stroke (width 0) (type default))
+  )
   (wire (pts (xy 185.42 132.08) (xy 215.9 132.08))
     (stroke (width 0) (type default))
@@
     (stroke (width 0) (type default))
   )
-  (wire (pts (xy 27.94 90.17) (xy 35.56 90.17))
-    (stroke (width 0) (type default))
-  )
   (wire (pts (xy 63.5 85.09) (xy 63.5 132.08))
     (stroke (width 0) (type default))
@@
     (stroke (width 0) (type default))
   )
+  (wire (pts (xy 54.61 99.06) (xy 54.61 58.42))
+    (stroke (width 0) (type default))
+  )
   (wire (pts (xy 99.06 101.6) (xy 99.06 106.68))
     (stroke (width 0) (type default))
@@
     (stroke (width 0) (type default))
   )
-  (wire (pts (xy 101.6 101.6) (xy 101.6 106.68))
+  (wire (pts (xy 101.6 99.06) (xy 101.6 106.68))
     (stroke (width 0) (type default))
   )
@@
     (stroke (width 0) (type default))
   )
-  (wire (pts (xy 49.53 40.64) (xy 49.53 43.18))
+  (wire (pts (xy 27.94 90.17) (xy 33.02 90.17))
     (stroke (width 0) (type default))
   )
@@
     (stroke (width 0) (type default))
   )
+  (wire (pts (xy 33.02 68.58) (xy 33.02 64.77))
+    (stroke (width 0) (type default))
+  )
+  (wire (pts (xy 27.94 58.42) (xy 35.56 58.42))
+    (stroke (width 0) (type default))
+  )
   (wire (pts (xy 54.61 46.99) (xy 105.41 46.99))
     (stroke (width 0) (type default))
   )
+  (wire (pts (xy 27.94 68.58) (xy 33.02 68.58))
+    (stroke (width 0) (type default))
+  )
   (wire (pts (xy 185.42 106.68) (xy 185.42 91.44))
     (stroke (width 0) (type default))
@@
     (stroke (width 0) (type default))
   )
-  (wire (pts (xy 27.94 58.42) (xy 33.02 58.42))
-    (stroke (width 0) (type default))
-  )
-  (wire (pts (xy 27.94 80.01) (xy 33.02 80.01))
-    (stroke (width 0) (type default))
-  )
   (wire (pts (xy 149.86 88.9) (xy 78.74 88.9))
     (stroke (width 0) (type default))
@@
     (stroke (width 0) (type default))
   )
+  (wire (pts (xy 27.94 80.01) (xy 35.56 80.01))
+    (stroke (width 0) (type default))
+  )
   (bus (pts (xy 198.12 121.92) (xy 198.12 124.46))
     (stroke (width 0) (type default))
   )
+  (wire (pts (xy 101.6 99.06) (xy 54.61 99.06))
+    (stroke (width 0) (type default))
+  )
   (wire (pts (xy 76.2 50.8) (xy 102.87 50.8))
     (stroke (width 0) (type default))
@@
     (stroke (width 0) (type default))
   )
-  (wire (pts (xy 35.56 68.58) (xy 35.56 64.77))
-    (stroke (width 0) (type default))
-  )
   (bus (pts (xy 82.55 82.55) (xy 72.39 82.55))
     (stroke (width 0) (type default))
@@
     (stroke (width 0) (type default))
   )
+  (wire (pts (xy 35.56 58.42) (xy 39.37 58.42))
+    (stroke (width 0) (type default))
+  )
   (wire (pts (xy 85.09 71.12) (xy 95.25 71.12))
     (stroke (width 0) (type default))
@@
     (stroke (width 0) (type default))
   )
-  (wire (pts (xy 54.61 40.64) (xy 54.61 46.99))
-    (stroke (width 0) (type default))
-  )
   (wire (pts (xy 27.94 71.12) (xy 30.48 71.12))
     (stroke (width 0) (type default))
@@
     (stroke (width 0) (type default))
   )
-  (wire (pts (xy 35.56 64.77) (xy 39.37 64.77))
-    (stroke (width 0) (type default))
-  )
   (wire (pts (xy 203.2 55.88) (xy 203.2 50.8))
     (stroke (width 0) (type default))
@@
   )
   (wire (pts (xy 205.74 55.88) (xy 205.74 48.26))
+    (stroke (width 0) (type default))
+  )
+  (wire (pts (xy 49.53 101.6) (xy 49.53 64.77))
     (stroke (width 0) (type default))
   )
@@
     )
   )
-  (hierarchical_label "12V0" (shape input) (at 54.61 40.64 90) (fields_autoplaced)
-    (effects (font (size 1.27 1.27)) (justify left))
-  )
-  (hierarchical_label "24V0" (shape input) (at 218.44 101.6 90) (fields_autoplaced)
-    (effects (font (size 1.27 1.27)) (justify left))
-  )
-  (hierarchical_label "12V0" (shape input) (at 101.6 101.6 90) (fields_autoplaced)
-    (effects (font (size 1.27 1.27)) (justify left))
-  )
   (hierarchical_label "GND" (shape input) (at 63.5 137.16 270) (fields_autoplaced)
     (effects (font (size 1.27 1.27)) (justify right))
-  )
-  (hierarchical_label "24V0" (shape input) (at 49.53 40.64 90) (fields_autoplaced)
-    (effects (font (size 1.27 1.27)) (justify left))
-  )
-  (hierarchical_label "24V0" (shape input) (at 99.06 101.6 90) (fields_autoplaced)
-    (effects (font (size 1.27 1.27)) (justify left))
   )
   (symbol (lib_id "Connector_Generic:Conn_01x02") (at 22.86 60.96 180) (unit 1)
@@
       (effects (font (size 1.27 1.27)) (justify left))
     )
-    (pin "24V0" input (at 218.44 106.68 90)
-      (effects (font (size 1.27 1.27)) (justify right))
-    )
     (instances
