File: rollo control.kicad_sch (KiCad schematic)
At the start: 1 part

Commit message: place
Parts:
- added VIC_EN1 (x2): Conn_01x02, Connector_Phoenix_MSTB:PhoenixContact_MSTBA_2,5_2-G-5,08_1x02_P5.08mm_Horizontal, symbol Connector_Generic:Conn_01x02
Connections:
- net 12V0: now also VIC_EN1.2 (Pin_2)
- net 24V0: now also VIC_EN1.2 (Pin_2)
- net Batt-: now also VIC_EN1.1 (Pin_1), VIC_EN1.1 (Pin_1)
Changed lines of the file:
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@@
 (kicad_sch (version 20230121) (generator eeschema)
   (paper "A4")
-  (bus_alias "Ain" (members "Ain_ntc+" "Ain_ntc-" "Ain_12V_Sig" "Ain_24V_Sig"))
-  (bus_alias "Stepper" (members "Step_step" "Step_dir" "Step_MS1" "Step_MS2" "Step_MS3" "Step_enable" "Step_sleep" "Step_reset"))
-  (bus_alias "DCDrive" (members "IFX1_FB" "IFX1_IN" "IFX1_INH" "IFX2_FB" "IFX2_IN" "IFX2_INH"))
-  (bus_alias "SolidState" (members "pump1" "pump2" "pump3" "pump4" "pump_fb2" "pump_fb1"))
   (bus_alias "Din" (members "I2C_SDA" "I2C_SCL" "FLW_Sig1" "FLW_Sig2" "BTN_1" "BTN_2" "ONE_SIG" ""))
   (bus_alias "Autoterm" (members "RX" "TX"))
   (bus_alias "485" (members "poci" "pico" "enable" ""))
+  (bus_alias "DCDrive" (members "IFX1_FB" "IFX1_IN" "IFX1_INH" "IFX2_FB" "IFX2_IN" "IFX2_INH"))
+  (bus_alias "SolidState" (members "pump1" "pump2" "pump3" "pump4" "pump_fb2" "pump_fb1"))
   (bus_alias "Rel" (members "REL1" "REL2" "REL3" "REL4" "REL5" "REL6" "REL7"))
+  (bus_alias "Stepper" (members "Step_step" "Step_dir" "Step_MS1" "Step_MS2" "Step_MS3" "Step_enable" "Step_sleep" "Step_reset"))
+  (bus_alias "Ain" (members "Ain_ntc+" "Ain_ntc-" "Ain_12V_Sig" "Ain_24V_Sig"))
   (junction (at 116.84 82.55) (diameter 0) (color 0 0 0 0)
   )
@@
   (junction (at 180.34 88.9) (diameter 0) (color 0 0 0 0)
   )
+  (junction (at 55.88 74.93) (diameter 0) (color 0 0 0 0)
+  )
   (junction (at 147.32 82.55) (diameter 0) (color 0 0 0 0)
   )
@@
   (junction (at 135.89 85.09) (diameter 0) (color 0 0 0 0)
   )
+  (junction (at 34.29 71.12) (diameter 0) (color 0 0 0 0)
+  )
   (junction (at 46.99 46.99) (diameter 0) (color 0 0 0 0)
   )
@@
     (stroke (width 0) (type default))
   )
+  (wire (pts (xy 34.29 74.93) (xy 55.88 74.93))
+    (stroke (width 0) (type default))
+  )
   (bus (pts (xy 116.84 82.55) (xy 109.22 82.55))
     (stroke (width 0) (type default))
@@
     (stroke (width 0) (type default))
   )
-  (wire (pts (xy 55.88 66.04) (xy 55.88 85.09))
+  (wire (pts (xy 55.88 66.04) (xy 55.88 74.93))
     (stroke (width 0) (type default))
   )
@@
     (stroke (width 0) (type default))
   )
+  (wire (pts (xy 34.29 71.12) (xy 34.29 74.93))
+    (stroke (width 0) (type default))
+  )
   (wire (pts (xy 67.31 111.76) (xy 80.01 111.76))
     (stroke (width 0) (type default))
@@
     (stroke (width 0) (type default))
   )
-  (wire (pts (xy 38.1 64.77) (xy 41.91 64.77))
+  (wire (pts (xy 31.75 64.77) (xy 41.91 64.77))
     (stroke (width 0) (type default))
   )
@@
     (stroke (width 0) (type default))
   )
+  (wire (pts (xy 27.94 68.58) (xy 31.75 68.58))
+    (stroke (width 0) (type default))
+  )
   (bus (pts (xy 152.4 82.55) (xy 180.34 82.55))
     (stroke (width 0) (type default))
@@
     (stroke (width 0) (type default))
   )
-  (wire (pts (xy 38.1 58.42) (xy 46.99 58.42))
+  (wire (pts (xy 27.94 58.42) (xy 46.99 58.42))
     (stroke (width 0) (type default))
   )
@@
     (stroke (width 0) (type default))
   )
+  (wire (pts (xy 31.75 68.58) (xy 31.75 64.77))
+    (stroke (width 0) (type default))
+  )
   (bus (pts (xy 74.93 82.55) (xy 64.77 82.55))
     (stroke (width 0) (type default))
@@
     (stroke (width 0) (type default))
   )
+  (wire (pts (xy 27.94 71.12) (xy 34.29 71.12))
+    (stroke (width 0) (type default))
+  )
   (wire (pts (xy 119.38 114.3) (xy 128.27 114.3))
     (stroke (width 0) (type default))
   )
+  (wire (pts (xy 55.88 74.93) (xy 55.88 85.09))
+    (stroke (width 0) (type default))
+  )
   (bus (pts (xy 147.32 62.23) (xy 147.32 64.77))
     (stroke (width 0) (type default))
@@
     (stroke (width 0) (type default))
   )
+  (wire (pts (xy 34.29 60.96) (xy 34.29 71.12))
+    (stroke (width 0) (type default))
+  )
   (wire (pts (xy 177.8 91.44) (xy 68.58 91.44))
     (stroke (width 0) (type default))
@@
   )
   (bus (pts (xy 190.5 124.46) (xy 190.5 127))
+    (stroke (width 0) (type default))
+  )
+  (wire (pts (xy 27.94 60.96) (xy 34.29 60.96))
     (stroke (width 0) (type default))
   )
@@
   (hierarchical_label "24V0" (shape input) (at 91.44 101.6 90) (fields_autoplaced)
     (effects (font (size 1.27 1.27)) (justify left))
+  )
+  (symbol (lib_id "Connector_Generic:Conn_01x02") (at 22.86 60.96 180) (unit 1)
+    (in_bom yes) (on_board yes) (dnp no)
+    (property "Reference" "VIC_EN1" (at 27.94 55.88 0)
+      (effects (font (size 1.27 1.27)) (justify left))
+    )
+    (property "Value" "Conn_01x02" (at 30.48 53.34 0)
+      (effects (font (size 1.27 1.27)) (justify left) hide)
+    )
+    (property "Footprint" "Connector_Phoenix_MSTB:PhoenixContact_MSTBA_2,5_2-G-5,08_1x02_P5.08mm_Horizontal" (at 22.86 60.96 0)
+      (effects (font (size 1.27 1.27)) hide)
+    )
+    (property "Datasheet" "~" (at 22.86 60.96 0)
+      (effects (font (size 1.27 1.27)) hide)
+    )
+    (pin "1")
+    (pin "2")
+    (instances
+      (project "rollo control"
+        (path "/7fd4875b-e2b3-49e9-a377-320ee6c6aef7/f84d4e41-04bc-49f0-bae3-d4cb51e0b9a0"
+          (reference "VIC_EN1") (unit 1)
+        )
+        (path "/7fd4875b-e2b3-49e9-a377-320ee6c6aef7/4e3087fc-fc79-4dc0-b9f3-dc50efd75935"
+          (reference "DCDRIVE1") (unit 1)
+        )
+        (path "/7fd4875b-e2b3-49e9-a377-320ee6c6aef7"
+          (reference "PWR_IN1") (unit 1)
+        )
+      )
+    )
   )
   (symbol (lib_id "Jumper:Jumper_2_Bridged") (at 55.88 91.44 270) (unit 1)
@@
         )
       )
+    )
+  )
+  (symbol (lib_id "Connector_Generic:Conn_01x02") (at 22.86 71.12 180) (unit 1)
+    (in_bom yes) (on_board yes) (dnp no)
+    (property "Reference" "VIC_EN1" (at 27.94 66.04 0)
+      (effects (font (size 1.27 1.27)) (justify left))
+    )
+    (property "Value" "Conn_01x02" (at 29.21 67.31 90)
+      (effects (font (size 1.27 1.27)) (justify left) hide)
+    )
+    (property "Footprint" "Connector_Phoenix_MSTB:PhoenixContact_MSTBA_2,5_2-G-5,08_1x02_P5.08mm_Horizontal" (at 22.86 71.12 0)
+      (effects (font (size 1.27 1.27)) hide)
+    )
+    (property "Datasheet" "~" (at 22.86 71.12 0)
+      (effects (font (size 1.27 1.27)) hide)
+    )
+    (pin "1")
+    (pin "2")
+    (instances
+      (project "rollo control"
+        (path "/7fd4875b-e2b3-49e9-a377-320ee6c6aef7/f84d4e41-04bc-49f0-bae3-d4cb51e0b9a0"
+          (reference "VIC_EN1") (unit 1)
+        )
+        (path "/7fd4875b-e2b3-49e9-a377-320ee6c6aef7/4e3087fc-fc79-4dc0-b9f3-dc50efd75935"
+          (reference "DCDRIVE1") (unit 1)
+        )
+        (path "/7fd4875b-e2b3-49e9-a377-320ee6c6aef7"
+          (reference "PWR_IN2") (unit 1)
+        )
+      )

Commit message: mc1.5
Other:
- sheet Analog-IN ports: added ntc0+, ntc0-, ntc1+, ntc1-; removed ntc+, ntc-
- sheet Autoterm ports: added 5V0; removed none
- sheet mcu-relais ports: added 24V0; removed none

Commit message: 605
Parts:
- added F2, F3: Fuse, Fuse:Fuseholder_Blade_ATO_Littelfuse_Pudenz_2_Pin, symbol Device:Fuse
Connections:
- net 12V0: now also F2.2; no longer VIC_EN1.2 (Pin_2)
- net 24V0: now also F3.2; no longer VIC_EN1.2 (Pin_2)
- new net: F2.1, VIC_EN1.2 (Pin_2)
- new net: F3.1, VIC_EN1.2 (Pin_2)
Changed lines of the file:
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@@
   (junction (at 142.24 132.08) (diameter 0) (color 0 0 0 0)
   )
+  (junction (at 30.48 71.12) (diameter 0) (color 0 0 0 0)
+  )
   (junction (at 180.34 82.55) (diameter 0) (color 0 0 0 0)
   )
@@
   (junction (at 135.89 85.09) (diameter 0) (color 0 0 0 0)
   )
-  (junction (at 34.29 71.12) (diameter 0) (color 0 0 0 0)
-  )
   (junction (at 46.99 46.99) (diameter 0) (color 0 0 0 0)
   )
@@
     (stroke (width 0) (type default))
   )
-  (wire (pts (xy 34.29 74.93) (xy 55.88 74.93))
+  (wire (pts (xy 30.48 74.93) (xy 55.88 74.93))
     (stroke (width 0) (type default))
   )
@@
     (stroke (width 0) (type default))
   )
-  (wire (pts (xy 34.29 71.12) (xy 34.29 74.93))
+  (wire (pts (xy 30.48 71.12) (xy 30.48 74.93))
     (stroke (width 0) (type default))
   )
@@
     (stroke (width 0) (type default))
   )
-  (wire (pts (xy 31.75 64.77) (xy 41.91 64.77))
-    (stroke (width 0) (type default))
-  )
   (wire (pts (xy 77.47 58.42) (xy 87.63 58.42))
     (stroke (width 0) (type default))
@@
     (stroke (width 0) (type default))
   )
-  (wire (pts (xy 27.94 58.42) (xy 46.99 58.42))
+  (wire (pts (xy 27.94 58.42) (xy 31.75 58.42))
     (stroke (width 0) (type default))
   )
@@
     (stroke (width 0) (type default))
   )
-  (wire (pts (xy 27.94 71.12) (xy 34.29 71.12))
+  (wire (pts (xy 27.94 71.12) (xy 30.48 71.12))
     (stroke (width 0) (type default))
   )
@@
     (stroke (width 0) (type default))
   )
+  (wire (pts (xy 39.37 64.77) (xy 41.91 64.77))
+    (stroke (width 0) (type default))
+  )
   (bus (pts (xy 147.32 62.23) (xy 147.32 64.77))
     (stroke (width 0) (type default))
@@
     (stroke (width 0) (type default))
   )
+  (wire (pts (xy 39.37 58.42) (xy 46.99 58.42))
+    (stroke (width 0) (type default))
+  )
   (wire (pts (xy 177.8 127) (xy 177.8 132.08))
     (stroke (width 0) (type default))
@@
     (stroke (width 0) (type default))
   )
-  (wire (pts (xy 34.29 60.96) (xy 34.29 71.12))
+  (wire (pts (xy 30.48 60.96) (xy 30.48 71.12))
     (stroke (width 0) (type default))
   )
@@
     (stroke (width 0) (type default))
   )
-  (wire (pts (xy 27.94 60.96) (xy 34.29 60.96))
+  (wire (pts (xy 27.94 60.96) (xy 30.48 60.96))
     (stroke (width 0) (type default))
   )
@@
     (effects (font (size 1.27 1.27)) (justify left bottom))
   )
-  (label "Ain_ntc0+" (at 68.58 114.3 0)
+  (label "Ain_ntc0+" (at 68.58 114.3 0) (fields_autoplaced)
     (effects (font (size 1.27 1.27)) (justify left bottom))
   )
@@
     (effects (font (size 1.27 1.27)) (justify left bottom))
   )
-  (label "Ain_ntc1-" (at 68.58 121.92 0)
+  (label "Ain_ntc1-" (at 68.58 121.92 0) (fields_autoplaced)
     (effects (font (size 1.27 1.27)) (justify left bottom))
   )
@@
     (effects (font (size 1.27 1.27)) (justify left bottom))
   )
-  (label "Ain_ntc0-" (at 68.58 116.84 0)
+  (label "Ain_ntc0-" (at 68.58 116.84 0) (fields_autoplaced)
     (effects (font (size 1.27 1.27)) (justify left bottom))
   )
@@
     (effects (font (size 1.27 1.27)) (justify left bottom))
   )
-  (label "Ain_ntc1+" (at 68.58 119.38 0)
+  (label "Ain_ntc1+" (at 68.58 119.38 0) (fields_autoplaced)
     (effects (font (size 1.27 1.27)) (justify left bottom))
   )
@@
         )
       )
+    )
+  )
+  (symbol (lib_id "Device:Fuse") (at 35.56 58.42 90) (unit 1)
+    (in_bom yes) (on_board yes) (dnp no) (fields_autoplaced)
+    (property "Reference" "F2" (at 35.56 53.34 90)
+      (effects (font (size 1.27 1.27)))
+    )
+    (property "Value" "Fuse" (at 35.56 55.88 90)
+      (effects (font (size 1.27 1.27)))
+    )
+    (property "Footprint" "Fuse:Fuseholder_Blade_ATO_Littelfuse_Pudenz_2_Pin" (at 35.56 60.198 90)
+      (effects (font (size 1.27 1.27)) hide)
+    )
+    (property "Datasheet" "https://www.distrelec.de/Web/Downloads/_t/ds/1786164_eng_ger_tds.pdf" (at 35.56 58.42 0)
+      (effects (font (size 1.27 1.27)) hide)
+    )
+    (pin "1")
+    (pin "2")
+    (instances
+      (project "rollo control"
+        (path "/7fd4875b-e2b3-49e9-a377-320ee6c6aef7"
+          (reference "F2") (unit 1)
+        )
+      )
+    )
+  )
+  (symbol (lib_id "Device:Fuse") (at 35.56 64.77 90) (unit 1)
+    (in_bom yes) (on_board yes) (dnp no) (fields_autoplaced)
+    (property "Reference" "F3" (at 35.56 59.69 90)
+      (effects (font (size 1.27 1.27)))
+    )
+    (property "Value" "Fuse" (at 35.56 62.23 90)
+      (effects (font (size 1.27 1.27)))
+    )
+    (property "Footprint" "Fuse:Fuseholder_Blade_ATO_Littelfuse_Pudenz_2_Pin" (at 35.56 66.548 90)
+      (effects (font (size 1.27 1.27)) hide)
+    )
+    (property "Datasheet" "https://www.distrelec.de/Web/Downloads/_t/ds/1786164_eng_ger_tds.pdf" (at 35.56 64.77 0)
+      (effects (font (size 1.27 1.27)) hide)
+    )
+    (pin "1")
+    (pin "2")
+    (instances
+      (project "rollo control"
+        (path "/7fd4875b-e2b3-49e9-a377-320ee6c6aef7"
+          (reference "F3") (unit 1)
+        )
+      )

Commit message: placing
Parts:
- removed JP1: Jumper_2_Bridged, symbol Jumper:Jumper_2_Bridged
- added VIC_EN1 (x2): Conn_01x02, Connector_Phoenix_MSTB:PhoenixContact_MSTBA_2,5_2-G-5,08_1x02_P5.08mm_Horizontal, symbol Connector_Generic:Conn_01x02
- F2, F3: footprint Fuse:Fuseholder_Blade_ATO_Littelfuse_Pudenz_2_Pin -> Fuse:Fuseholder_Clip-5x20mm_Littelfuse_100_Inline_P20.50x4.60mm_D1.30mm_Horizontal
Connections:
- net Batt- is gone; now on net GND: VIC_EN1.1 (Pin_1), VIC_EN1.1 (Pin_1)
- net GND: now also VIC_EN1.1 (Pin_1), VIC_EN1.1 (Pin_1)
- net at F2.1, VIC_EN1.2 (Pin_2): now also VIC_EN1.2 (Pin_2)
- net at F3.1, VIC_EN1.2 (Pin_2): now also VIC_EN1.2 (Pin_2)
Other:
- moved on the sheet: F2

Commit message: dgfg
Other:
- removed sheet Stepper
Changed lines of the file:
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@@
-    )
-  )
-  (sheet (at 95.25 55.88) (size 15.24 22.86)
-    (stroke (width 0.1524) (type solid))
-    (fill (color 0 0 0 0.0000))
-    (property "Sheetname" "Stepper" (at 95.25 55.1684 0)
-      (effects (font (size 1.27 1.27)) (justify left bottom))
-    )
-    (property "Sheetfile" "A4988Stepper.kicad_sch" (at 95.25 79.3246 0)
-      (effects (font (size 1.27 1.27)) (justify left top) hide)
-    )
-    (property "Current" "2A" (at 100.33 80.01 0) (show_name)
-      (effects (font (size 1.27 1.27)))
-    )
-    (pin "3V3" input (at 102.87 55.88 90)
-      (effects (font (size 1.27 1.27)) (justify right))
-    )
-    (pin "MS3" input (at 95.25 68.58 180)
-      (effects (font (size 1.27 1.27)) (justify left))
-    )
-    (pin "dir" input (at 95.25 60.96 180)
-      (effects (font (size 1.27 1.27)) (justify left))
-    )
-    (pin "MS1" input (at 95.25 63.5 180)
-      (effects (font (size 1.27 1.27)) (justify left))
-    )
-    (pin "MS2" input (at 95.25 66.04 180)
-      (effects (font (size 1.27 1.27)) (justify left))
-    )
-    (pin "12V0" input (at 105.41 55.88 90)
-      (effects (font (size 1.27 1.27)) (justify right))
-    )
-    (pin "24V0" input (at 107.95 55.88 90)
-      (effects (font (size 1.27 1.27)) (justify right))
-    )
-    (pin "enable" input (at 95.25 71.12 180)
-      (effects (font (size 1.27 1.27)) (justify left))
-    )
-    (pin "sleep" input (at 95.25 73.66 180)
-      (effects (font (size 1.27 1.27)) (justify left))
-    )
-    (pin "step" input (at 95.25 58.42 180)
-      (effects (font (size 1.27 1.27)) (justify left))
-    )
-    (pin "reset" input (at 95.25 76.2 180)
-      (effects (font (size 1.27 1.27)) (justify left))
-    )
-    (pin "GND" input (at 107.95 78.74 270)
-      (effects (font (size 1.27 1.27)) (justify left))
-    )
-    (instances
-      (project "rollo control"
-        (path "/7fd4875b-e2b3-49e9-a377-320ee6c6aef7" (page "6"))
-      )
     )
   )

Commit message: gsdfg
dyfg
Parts:
- removed F3: Fuse, Fuse:Fuseholder_Clip-5x20mm_Littelfuse_100_Inline_P20.50x4.60mm_D1.30mm_Horizontal, symbol Device:Fuse
- removed VIC_EN1 (x2): Conn_01x02, Connector_Phoenix_MSTB:PhoenixContact_MSTBA_2,5_2-G-5,08_1x02_P5.08mm_Horizontal, symbol Connector_Generic:Conn_01x02
Other:
- sheet Analog-IN ports: added none; removed 24V0, 24V_SIG
- sheet DC Power ports: added none; removed 24V0
- sheet DCDrive ports: added none; removed 24V0
- sheet SolidState ports: added none; removed 24V0
- sheet mcu-relais ports: added none; removed 24V0
