File: relaisausgaenge.kicad_sch (KiCad schematic)
At the start: 8 parts, among them K1 TIANBO-HJR-4102-L, K2 TIANBO-HJR-4102-L, K3 TIANBO-HJR-4102-L, U7 ULN2004A

Commit message: place
Parts:
- U6: renamed from U7; footprint (none) -> Package_SO:TSSOP-16_4.4x5mm_P0.65mm
Changed lines of the file:
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@@
   (symbol (lib_id "Transistor_Array:ULN2004A") (at 76.2 90.17 0) (unit 1)
     (in_bom yes) (on_board yes) (dnp no) (fields_autoplaced)
-    (property "Reference" "U7" (at 76.2 74.4601 0)
+    (property "Reference" "U6" (at 76.2 74.4601 0)
       (effects (font (size 1.27 1.27)))
     )
@@
       (effects (font (size 1.27 1.27)))
     )
-    (property "Footprint" "" (at 77.47 104.14 0)
+    (property "Footprint" "Package_SO:TSSOP-16_4.4x5mm_P0.65mm" (at 77.47 104.14 0)
       (effects (font (size 1.27 1.27)) (justify left) hide)
     )
@@
       (project "rollo control"
         (path "/7fd4875b-e2b3-49e9-a377-320ee6c6aef7/f84d4e41-04bc-49f0-bae3-d4cb51e0b9a0"
-          (reference "U7") (unit 1)
+          (reference "U6") (unit 1)
         )
       )

Commit message: mc1.5
Parts:
- added JP10: Jumper_3_Bridged12, Connector_PinHeader_2.54mm:PinHeader_1x03_P2.54mm_Vertical, symbol Jumper:Jumper_3_Bridged12
Connections:
- net 5V0: now also JP10.1 (A); no longer EXT_REL_CON1.1 (Pin_1), K1.8, K2.8, K3.8, U6.9 (COM)
- new net: EXT_REL_CON1.1 (Pin_1), JP10.2 (C), K1.8, K2.8, K3.8, U6.9 (COM)
- new net 24V0: JP10.3 (B)
Changed lines of the file:
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@@
 (kicad_sch (version 20230121) (generator eeschema)
   (paper "A4")
+  (junction (at 165.1 80.01) (diameter 0) (color 0 0 0 0)
+  )
+  (junction (at 165.1 105.41) (diameter 0) (color 0 0 0 0)
+  )
+  (junction (at 91.44 80.01) (diameter 0) (color 0 0 0 0)
+  )
+  (junction (at 144.78 115.57) (diameter 0) (color 0 0 0 0)
+  )
   (wire (pts (xy 104.14 127) (xy 148.59 127))
     (stroke (width 0) (type default))
@@
     (stroke (width 0) (type default))
   )
+  (wire (pts (xy 91.44 115.57) (xy 91.44 80.01))
+    (stroke (width 0) (type default))
+  )
   (wire (pts (xy 109.22 90.17) (xy 109.22 105.41))
     (stroke (width 0) (type default))
@@
     (stroke (width 0) (type default))
   )
+  (wire (pts (xy 144.78 115.57) (xy 91.44 115.57))
+    (stroke (width 0) (type default))
+  )
+  (wire (pts (xy 161.29 105.41) (xy 165.1 105.41))
+    (stroke (width 0) (type default))
+  )
+  (wire (pts (xy 165.1 105.41) (xy 165.1 115.57))
+    (stroke (width 0) (type default))
+  )
   (wire (pts (xy 109.22 80.01) (xy 146.05 80.01))
     (stroke (width 0) (type default))
@@
     (stroke (width 0) (type default))
   )
+  (wire (pts (xy 91.44 74.93) (xy 91.44 80.01))
+    (stroke (width 0) (type default))
+  )
   (wire (pts (xy 106.68 92.71) (xy 106.68 124.46))
     (stroke (width 0) (type default))
   )
+  (wire (pts (xy 161.29 80.01) (xy 165.1 80.01))
+    (stroke (width 0) (type default))
+  )
   (wire (pts (xy 99.06 132.08) (xy 99.06 100.33))
     (stroke (width 0) (type default))
@@
     (stroke (width 0) (type default))
   )
-  (wire (pts (xy 86.36 80.01) (xy 92.71 80.01))
+  (wire (pts (xy 86.36 80.01) (xy 91.44 80.01))
     (stroke (width 0) (type default))
   )
@@
     (stroke (width 0) (type default))
   )
+  (wire (pts (xy 78.74 71.12) (xy 85.09 71.12))
+    (stroke (width 0) (type default))
+  )
   (wire (pts (xy 104.14 95.25) (xy 104.14 127))
     (stroke (width 0) (type default))
@@
     (stroke (width 0) (type default))
   )
+  (wire (pts (xy 165.1 80.01) (xy 165.1 105.41))
+    (stroke (width 0) (type default))
+  )
   (wire (pts (xy 161.29 44.45) (xy 175.26 44.45))
     (stroke (width 0) (type default))
@@
     (stroke (width 0) (type default))
   )
+  (wire (pts (xy 161.29 54.61) (xy 165.1 54.61))
+    (stroke (width 0) (type default))
+  )
   (wire (pts (xy 76.2 105.41) (xy 76.2 109.22))
     (stroke (width 0) (type default))
@@
     (stroke (width 0) (type default))
   )
+  (wire (pts (xy 97.79 71.12) (xy 100.33 71.12))
+    (stroke (width 0) (type default))
+  )
   (wire (pts (xy 106.68 54.61) (xy 146.05 54.61))
     (stroke (width 0) (type default))
   )
+  (wire (pts (xy 165.1 115.57) (xy 144.78 115.57))
+    (stroke (width 0) (type default))
+  )
+  (wire (pts (xy 144.78 115.57) (xy 144.78 121.92))
+    (stroke (width 0) (type default))
+  )
   (wire (pts (xy 170.18 41.91) (xy 175.26 41.91))
     (stroke (width 0) (type default))
   )
+  (wire (pts (xy 165.1 54.61) (xy 165.1 80.01))
+    (stroke (width 0) (type default))
+  )
   (wire (pts (xy 138.43 36.83) (xy 170.18 36.83))
     (stroke (width 0) (type default))
@@
     (stroke (width 0) (type default))
   )
+  (hierarchical_label "24V0" (shape input) (at 100.33 71.12 0) (fields_autoplaced)
+    (effects (font (size 1.27 1.27)) (justify left))
+  )
   (hierarchical_label "REL2" (shape input) (at 66.04 87.63 180) (fields_autoplaced)
     (effects (font (size 1.27 1.27)) (justify right))
   )
-  (hierarchical_label "5V0" (shape input) (at 161.29 80.01 0) (fields_autoplaced)
-    (effects (font (size 1.27 1.27)) (justify left))
-  )
   (hierarchical_label "REL7" (shape input) (at 66.04 100.33 180) (fields_autoplaced)
     (effects (font (size 1.27 1.27)) (justify right))
   )
-  (hierarchical_label "5V0" (shape input) (at 161.29 105.41 0) (fields_autoplaced)
-    (effects (font (size 1.27 1.27)) (justify left))
-  )
-  (hierarchical_label "5V0" (shape input) (at 92.71 80.01 0) (fields_autoplaced)
-    (effects (font (size 1.27 1.27)) (justify left))
-  )
   (hierarchical_label "GND" (shape input) (at 148.59 134.62 180) (fields_autoplaced)
     (effects (font (size 1.27 1.27)) (justify right))
@@
     (effects (font (size 1.27 1.27)) (justify right))
   )
-  (hierarchical_label "5V0" (shape input) (at 144.78 121.92 180) (fields_autoplaced)
+  (hierarchical_label "5V0" (shape input) (at 78.74 71.12 180) (fields_autoplaced)
     (effects (font (size 1.27 1.27)) (justify right))
   )
@@
   (hierarchical_label "GND" (shape input) (at 76.2 109.22 270) (fields_autoplaced)
     (effects (font (size 1.27 1.27)) (justify right))
-  )
-  (hierarchical_label "5V0" (shape input) (at 161.29 54.61 0) (fields_autoplaced)
-    (effects (font (size 1.27 1.27)) (justify left))
   )
   (hierarchical_label "REL1" (shape input) (at 66.04 85.09 180) (fields_autoplaced)
@@
         )
       )
+    )
+  )
+  (symbol (lib_id "Jumper:Jumper_3_Bridged12") (at 91.44 71.12 0) (unit 1)
+    (in_bom yes) (on_board yes) (dnp no) (fields_autoplaced)
+    (property "Reference" "JP10" (at 91.44 67.2459 0)
+      (effects (font (size 1.27 1.27)))
+    )
+    (property "Value" "Jumper_3_Bridged12" (at 91.44 69.1669 0)
+      (effects (font (size 1.27 1.27)))
+    )
+    (property "Footprint" "Connector_PinHeader_2.54mm:PinHeader_1x03_P2.54mm_Vertical" (at 91.44 71.12 0)
+      (effects (font (size 1.27 1.27)) hide)
+    )
+    (property "Datasheet" "~" (at 91.44 71.12 0)
+      (effects (font (size 1.27 1.27)) hide)
+    )
+    (pin "1")
+    (pin "2")
+    (pin "3")
+    (instances
+      (project "rollo control"
+        (path "/7fd4875b-e2b3-49e9-a377-320ee6c6aef7/42cd8867-79f6-4c26-8217-42f6d2cc80dc"
+          (reference "JP10") (unit 1)
+        )
+        (path "/7fd4875b-e2b3-49e9-a377-320ee6c6aef7/f84d4e41-04bc-49f0-bae3-d4cb51e0b9a0"
+          (reference "JP7") (unit 1)
+        )
+      )

Commit message: placing
Parts:
- VIC_EN1, VIC_EN2, VIC_EN3: footprint Connector_Phoenix_MSTB:PhoenixContact_MSTBA_2,5_2-G-5,08_1x02_P5.08mm_Horizontal -> Connector_Phoenix_MC:PhoenixContact_MC_1,5_2-G-3.5_1x02_P3.50mm_Horizontal
Other:
- moved on the sheet: EXT_REL_CON1
Changed lines of the file:
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@@
   (junction (at 91.44 80.01) (diameter 0) (color 0 0 0 0)
   )
-  (junction (at 144.78 115.57) (diameter 0) (color 0 0 0 0)
-  )
-  (wire (pts (xy 104.14 127) (xy 148.59 127))
+  (junction (at 165.1 115.57) (diameter 0) (color 0 0 0 0)
+  )
+  (wire (pts (xy 104.14 127) (xy 175.26 127))
     (stroke (width 0) (type default))
   )
@@
     (stroke (width 0) (type default))
   )
-  (wire (pts (xy 144.78 115.57) (xy 91.44 115.57))
+  (wire (pts (xy 91.44 115.57) (xy 165.1 115.57))
     (stroke (width 0) (type default))
   )
@@
     (stroke (width 0) (type default))
   )
+  (wire (pts (xy 175.26 134.62) (xy 148.59 134.62))
+    (stroke (width 0) (type default))
+  )
   (wire (pts (xy 86.36 95.25) (xy 104.14 95.25))
     (stroke (width 0) (type default))
@@
     (stroke (width 0) (type default))
   )
-  (wire (pts (xy 144.78 121.92) (xy 148.59 121.92))
+  (wire (pts (xy 165.1 121.92) (xy 175.26 121.92))
     (stroke (width 0) (type default))
   )
@@
     (stroke (width 0) (type default))
   )
-  (wire (pts (xy 148.59 124.46) (xy 106.68 124.46))
-    (stroke (width 0) (type default))
-  )
-  (wire (pts (xy 148.59 129.54) (xy 101.6 129.54))
+  (wire (pts (xy 175.26 124.46) (xy 106.68 124.46))
+    (stroke (width 0) (type default))
+  )
+  (wire (pts (xy 175.26 129.54) (xy 101.6 129.54))
     (stroke (width 0) (type default))
   )
@@
     (stroke (width 0) (type default))
   )
-  (wire (pts (xy 148.59 132.08) (xy 99.06 132.08))
+  (wire (pts (xy 175.26 132.08) (xy 99.06 132.08))
     (stroke (width 0) (type default))
   )
@@
     (stroke (width 0) (type default))
   )
-  (wire (pts (xy 165.1 115.57) (xy 144.78 115.57))
-    (stroke (width 0) (type default))
-  )
-  (wire (pts (xy 144.78 115.57) (xy 144.78 121.92))
+  (wire (pts (xy 165.1 115.57) (xy 165.1 121.92))
     (stroke (width 0) (type default))
   )
@@
     )
   )
-  (symbol (lib_id "Connector_Generic:Conn_01x06") (at 153.67 127 0) (unit 1)
-    (in_bom yes) (on_board yes) (dnp no) (fields_autoplaced)
-    (property "Reference" "EXT_REL_CON1" (at 155.702 127.6263 0)
-      (effects (font (size 1.27 1.27)) (justify left))
-    )
-    (property "Value" "Conn_01x06" (at 155.702 129.5473 0)
-      (effects (font (size 1.27 1.27)) (justify left))
-    )
-    (property "Footprint" "Connector_JST:JST_XH_B5B-XH-A_1x05_P2.50mm_Vertical" (at 153.67 127 0)
-      (effects (font (size 1.27 1.27)) hide)
-    )
-    (property "Datasheet" "~" (at 153.67 127 0)
+  (symbol (lib_id "Connector_Generic:Conn_01x06") (at 180.34 127 0) (unit 1)
+    (in_bom yes) (on_board yes) (dnp no) (fields_autoplaced)
+    (property "Reference" "EXT_REL_CON1" (at 182.372 127.6263 0)
+      (effects (font (size 1.27 1.27)) (justify left))
+    )
+    (property "Value" "Conn_01x06" (at 182.372 129.5473 0)
+      (effects (font (size 1.27 1.27)) (justify left))
+    )
+    (property "Footprint" "Connector_JST:JST_XH_B5B-XH-A_1x05_P2.50mm_Vertical" (at 180.34 127 0)
+      (effects (font (size 1.27 1.27)) hide)
+    )
+    (property "Datasheet" "~" (at 180.34 127 0)
       (effects (font (size 1.27 1.27)) hide)
     )
@@
       (effects (font (size 1.27 1.27)) (justify left))
     )
-    (property "Footprint" "Connector_Phoenix_MSTB:PhoenixContact_MSTBA_2,5_2-G-5,08_1x02_P5.08mm_Horizontal" (at 180.34 41.91 0)
+    (property "Footprint" "Connector_Phoenix_MC:PhoenixContact_MC_1,5_2-G-3.5_1x02_P3.50mm_Horizontal" (at 180.34 41.91 0)
       (effects (font (size 1.27 1.27)) hide)
     )
@@
       (effects (font (size 1.27 1.27)) (justify left))
     )
-    (property "Footprint" "Connector_Phoenix_MSTB:PhoenixContact_MSTBA_2,5_2-G-5,08_1x02_P5.08mm_Horizontal" (at 180.34 92.71 0)
+    (property "Footprint" "Connector_Phoenix_MC:PhoenixContact_MC_1,5_2-G-3.5_1x02_P3.50mm_Horizontal" (at 180.34 92.71 0)
       (effects (font (size 1.27 1.27)) hide)
     )
@@
       (effects (font (size 1.27 1.27)) (justify left))
     )
-    (property "Footprint" "Connector_Phoenix_MSTB:PhoenixContact_MSTBA_2,5_2-G-5,08_1x02_P5.08mm_Horizontal" (at 180.34 67.31 0)
-      (effects (font (size 1.27 1.27)) hide)
-    )
+    (property "Footprint" "Connector_Phoenix_MC:PhoenixContact_MC_1,5_2-G-3.5_1x02_P3.50mm_Horizontal" (at 180.34 67.31 0)
+      (effects (font (size 1.27 1.27)) hide)
+    )

Commit message: placing2
Parts:
- removed JP10: Jumper_3_Bridged12, Connector_PinHeader_2.54mm:PinHeader_1x03_P2.54mm_Vertical, symbol Jumper:Jumper_3_Bridged12
Connections:
- net 5V0: now also EXT_REL_CON1.1 (Pin_1), K1.8, K2.8, K3.8, U6.9 (COM)
Changed lines of the file:
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@@
     (stroke (width 0) (type default))
   )
-  (wire (pts (xy 91.44 74.93) (xy 91.44 80.01))
+  (wire (pts (xy 91.44 71.12) (xy 91.44 80.01))
     (stroke (width 0) (type default))
   )
@@
     (stroke (width 0) (type default))
   )
-  (wire (pts (xy 78.74 71.12) (xy 85.09 71.12))
+  (wire (pts (xy 78.74 71.12) (xy 91.44 71.12))
     (stroke (width 0) (type default))
   )
@@
     (stroke (width 0) (type default))
   )
-  (wire (pts (xy 97.79 71.12) (xy 100.33 71.12))
-    (stroke (width 0) (type default))
-  )
   (wire (pts (xy 106.68 54.61) (xy 146.05 54.61))
     (stroke (width 0) (type default))
@@
   (wire (pts (xy 171.45 67.31) (xy 175.26 67.31))
     (stroke (width 0) (type default))
-  )
-  (hierarchical_label "24V0" (shape input) (at 100.33 71.12 0) (fields_autoplaced)
-    (effects (font (size 1.27 1.27)) (justify left))
   )
   (hierarchical_label "REL2" (shape input) (at 66.04 87.63 180) (fields_autoplaced)
@@
         )
       )
-    )
-  )
-  (symbol (lib_id "Jumper:Jumper_3_Bridged12") (at 91.44 71.12 0) (unit 1)
-    (in_bom yes) (on_board yes) (dnp no) (fields_autoplaced)
-    (property "Reference" "JP10" (at 91.44 67.2459 0)
-      (effects (font (size 1.27 1.27)))
-    )
-    (property "Value" "Jumper_3_Bridged12" (at 91.44 69.1669 0)
-      (effects (font (size 1.27 1.27)))
-    )
-    (property "Footprint" "Connector_PinHeader_2.54mm:PinHeader_1x03_P2.54mm_Vertical" (at 91.44 71.12 0)
-      (effects (font (size 1.27 1.27)) hide)
-    )
-    (property "Datasheet" "~" (at 91.44 71.12 0)
-      (effects (font (size 1.27 1.27)) hide)
-    )
-    (pin "1")
-    (pin "2")
-    (pin "3")
-    (instances
-      (project "rollo control"
-        (path "/7fd4875b-e2b3-49e9-a377-320ee6c6aef7/42cd8867-79f6-4c26-8217-42f6d2cc80dc"
-          (reference "JP10") (unit 1)
-        )
-        (path "/7fd4875b-e2b3-49e9-a377-320ee6c6aef7/f84d4e41-04bc-49f0-bae3-d4cb51e0b9a0"
-          (reference "JP7") (unit 1)
-        )
-      )

Commit message: gsdfg
dyfg
Parts:
- removed K1, K2, K3: TIANBO-HJR-4102-L, Relay_THT:Relay_SPDT_HJR-4102, symbol Relay:TIANBO-HJR-4102-L
- removed VIC_EN1, VIC_EN2, VIC_EN3: Conn_01x02, Connector_Phoenix_MC:PhoenixContact_MC_1,5_2-G-3.5_1x02_P3.50mm_Horizontal, symbol Connector_Generic:Conn_01x02
- added EXT_REL_CON2: Conn_01x06, Connector_JST:JST_XH_B5B-XH-A_1x05_P2.50mm_Vertical, symbol Connector_Generic:Conn_01x06
Connections:
- net 5V0: now also EXT_REL_CON2.1 (Pin_1)
- net GND: now also EXT_REL_CON2.6 (Pin_6)
- net at U6.14 (O3): now also EXT_REL_CON2.5 (Pin_5)
- net at U6.15 (O2): now also EXT_REL_CON2.4 (Pin_4)
- net at U6.16 (O1): now also EXT_REL_CON2.3 (Pin_3)
