File: uart level shifter.kicad_sch (KiCad schematic)
At the start: 5 parts, among them U9 TXB0104PW

Commit message: place
Parts:
- renumbered U9 to U8, UART_AUTOTERM to UART_AUTOTERM1
Changed lines of the file:
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@@
   (symbol (lib_id "Connector_Generic:Conn_01x04") (at 163.83 64.77 0) (unit 1)
     (in_bom yes) (on_board yes) (dnp no) (fields_autoplaced)
-    (property "Reference" "UART_AUTOTERM" (at 166.37 64.77 0)
+    (property "Reference" "UART_AUTOTERM1" (at 166.37 64.77 0)
       (effects (font (size 1.27 1.27)) (justify left))
     )
@@
       (project "rollo control"
         (path "/7fd4875b-e2b3-49e9-a377-320ee6c6aef7/42cd8867-79f6-4c26-8217-42f6d2cc80dc"
-          (reference "UART_AUTOTERM") (unit 1)
+          (reference "UART_AUTOTERM1") (unit 1)
         )
       )
@@
   (symbol (lib_id "Logic_LevelTranslator:TXB0104PW") (at 116.84 72.39 0) (unit 1)
     (in_bom yes) (on_board yes) (dnp no) (fields_autoplaced)
-    (property "Reference" "U9" (at 118.7959 90.17 0)
+    (property "Reference" "U8" (at 118.7959 90.17 0)
       (effects (font (size 1.27 1.27)) (justify left))
     )
@@
       (project "rollo control"
         (path "/7fd4875b-e2b3-49e9-a377-320ee6c6aef7/42cd8867-79f6-4c26-8217-42f6d2cc80dc"
-          (reference "U9") (unit 1)
+          (reference "U8") (unit 1)
         )
       )

Commit message: mc1.5
Parts:
- added C33: C_Small, symbol Device:C_Small
- added JP10: Jumper_3_Bridged12, Connector_PinHeader_2.54mm:PinHeader_1x03_P2.54mm_Vertical, symbol Jumper:Jumper_3_Bridged12
Connections:
- net 3V3: now also JP10.1 (A)
- net GND: now also UART_AUTOTERM1.2 (Pin_2), C33.2; no longer UART_AUTOTERM1.4 (Pin_4)
- net at D1.1 (K), U8.12 (B2): now also UART_AUTOTERM1.4 (Pin_4); no longer UART_AUTOTERM1.3 (Pin_3)
- net at D1.2 (K), U8.13 (B1): now also UART_AUTOTERM1.3 (Pin_3); no longer UART_AUTOTERM1.2 (Pin_2)
- net at C32.1, U8.14 (VCCB), UART_AUTOTERM1.1 (Pin_1): now also JP10.2 (C)
- new net 5V0: C33.1, JP10.3 (B)
Other:
- note added: "Connector_JST:JST_XH_B5B-XH-A_1x05_P2.50mm_Vertical"
- moved on the sheet: UART_AUTOTERM1
Changed lines of the file:
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@@
 (kicad_sch (version 20230121) (generator eeschema)
   (paper "A4")
+  (junction (at 114.3 48.26) (diameter 0) (color 0 0 0 0)
+  )
+  (junction (at 142.24 64.77) (diameter 0) (color 0 0 0 0)
+  )
   (junction (at 139.7 90.17) (diameter 0) (color 0 0 0 0)
   )
-  (junction (at 142.24 64.77) (diameter 0) (color 0 0 0 0)
+  (junction (at 156.21 52.07) (diameter 0) (color 0 0 0 0)
   )
   (junction (at 116.84 90.17) (diameter 0) (color 0 0 0 0)
@@
   (junction (at 114.3 38.1) (diameter 0) (color 0 0 0 0)
   )
+  (junction (at 162.56 36.83) (diameter 0) (color 0 0 0 0)
+  )
   (junction (at 137.16 69.85) (diameter 0) (color 0 0 0 0)
   )
@@
     (stroke (width 0) (type default))
   )
+  (wire (pts (xy 142.24 64.77) (xy 142.24 73.66))
+    (stroke (width 0) (type default))
+  )
   (wire (pts (xy 137.16 73.66) (xy 137.16 69.85))
     (stroke (width 0) (type default))
   )
-  (wire (pts (xy 114.3 38.1) (xy 114.3 54.61))
-    (stroke (width 0) (type default))
-  )
   (wire (pts (xy 96.52 64.77) (xy 106.68 64.77))
     (stroke (width 0) (type default))
   )
-  (wire (pts (xy 156.21 69.85) (xy 158.75 69.85))
-    (stroke (width 0) (type default))
-  )
   (wire (pts (xy 116.84 90.17) (xy 116.84 96.52))
     (stroke (width 0) (type default))
   )
+  (wire (pts (xy 162.56 36.83) (xy 162.56 48.26))
+    (stroke (width 0) (type default))
+  )
+  (wire (pts (xy 173.99 36.83) (xy 173.99 38.1))
+    (stroke (width 0) (type default))
+  )
   (wire (pts (xy 114.3 38.1) (xy 120.65 38.1))
     (stroke (width 0) (type default))
   )
+  (wire (pts (xy 134.62 52.07) (xy 156.21 52.07))
+    (stroke (width 0) (type default))
+  )
+  (wire (pts (xy 114.3 48.26) (xy 114.3 54.61))
+    (stroke (width 0) (type default))
+  )
+  (wire (pts (xy 156.21 67.31) (xy 156.21 69.85))
+    (stroke (width 0) (type default))
+  )
+  (wire (pts (xy 173.99 36.83) (xy 162.56 36.83))
+    (stroke (width 0) (type default))
+  )
+  (wire (pts (xy 114.3 38.1) (xy 114.3 48.26))
+    (stroke (width 0) (type default))
+  )
+  (wire (pts (xy 156.21 67.31) (xy 158.75 67.31))
+    (stroke (width 0) (type default))
+  )
+  (wire (pts (xy 156.21 59.69) (xy 156.21 52.07))
+    (stroke (width 0) (type default))
+  )
+  (wire (pts (xy 158.75 62.23) (xy 152.4 62.23))
+    (stroke (width 0) (type default))
+  )
   (wire (pts (xy 142.24 64.77) (xy 158.75 64.77))
     (stroke (width 0) (type default))
   )
-  (wire (pts (xy 134.62 52.07) (xy 156.21 52.07))
-    (stroke (width 0) (type default))
-  )
-  (wire (pts (xy 137.16 67.31) (xy 137.16 69.85))
-    (stroke (width 0) (type default))
-  )
-  (wire (pts (xy 156.21 62.23) (xy 156.21 52.07))
-    (stroke (width 0) (type default))
-  )
-  (wire (pts (xy 156.21 90.17) (xy 156.21 69.85))
-    (stroke (width 0) (type default))
-  )
   (wire (pts (xy 119.38 52.07) (xy 134.62 52.07))
     (stroke (width 0) (type default))
   )
-  (wire (pts (xy 139.7 90.17) (xy 156.21 90.17))
+  (wire (pts (xy 139.7 90.17) (xy 152.4 90.17))
     (stroke (width 0) (type default))
   )
@@
     (stroke (width 0) (type default))
   )
-  (wire (pts (xy 142.24 64.77) (xy 142.24 73.66))
-    (stroke (width 0) (type default))
-  )
   (wire (pts (xy 127 64.77) (xy 142.24 64.77))
     (stroke (width 0) (type default))
   )
+  (wire (pts (xy 162.56 34.29) (xy 162.56 36.83))
+    (stroke (width 0) (type default))
+  )
   (wire (pts (xy 96.52 69.85) (xy 106.68 69.85))
     (stroke (width 0) (type default))
   )
-  (wire (pts (xy 158.75 67.31) (xy 137.16 67.31))
+  (wire (pts (xy 114.3 48.26) (xy 149.86 48.26))
     (stroke (width 0) (type default))
   )
@@
     (stroke (width 0) (type default))
   )
-  (wire (pts (xy 158.75 62.23) (xy 156.21 62.23))
-    (stroke (width 0) (type default))
+  (wire (pts (xy 156.21 69.85) (xy 137.16 69.85))
+    (stroke (width 0) (type default))
+  )
+  (wire (pts (xy 152.4 62.23) (xy 152.4 90.17))
+    (stroke (width 0) (type default))
+  )
+  (wire (pts (xy 158.75 59.69) (xy 156.21 59.69))
+    (stroke (width 0) (type default))
+  )
+  (text "Connector_JST:JST_XH_B5B-XH-A_1x05_P2.50mm_Vertical"
+    (at 200.66 55.88 0)
+    (effects (font (size 1.27 1.27)) (justify left bottom))
   )
   (hierarchical_label "RX" (shape input) (at 96.52 64.77 180) (fields_autoplaced)
@@
     (effects (font (size 1.27 1.27)) (justify right))
   )
+  (hierarchical_label "5V0" (shape input) (at 162.56 34.29 90) (fields_autoplaced)
+    (effects (font (size 1.27 1.27)) (justify left))
+  )
+  (hierarchical_label "GND" (shape input) (at 173.99 43.18 270) (fields_autoplaced)
+    (effects (font (size 1.27 1.27)) (justify right))
+  )
   (hierarchical_label "GND" (shape input) (at 120.65 43.18 270) (fields_autoplaced)
     (effects (font (size 1.27 1.27)) (justify right))
   )
+  (symbol (lib_id "Device:C_Small") (at 173.99 40.64 0) (mirror y) (unit 1)
+    (in_bom yes) (on_board yes) (dnp no) (fields_autoplaced)
+    (property "Reference" "C33" (at 171.45 39.3763 0)
+      (effects (font (size 1.27 1.27)) (justify left))
+    )
+    (property "Value" "C_Small" (at 171.45 41.9163 0)
+      (effects (font (size 1.27 1.27)) (justify left))
+    )
+    (property "Footprint" "" (at 173.99 40.64 0)
+      (effects (font (size 1.27 1.27)) hide)
+    )
+    (property "Datasheet" "~" (at 173.99 40.64 0)
+      (effects (font (size 1.27 1.27)) hide)
+    )
+    (pin "1")
+    (pin "2")
+    (instances
+      (project "rollo control"
+        (path "/7fd4875b-e2b3-49e9-a377-320ee6c6aef7/42cd8867-79f6-4c26-8217-42f6d2cc80dc"
+          (reference "C33") (unit 1)
+        )
+      )
+    )
+  )
   (symbol (lib_id "Device:C_Small") (at 120.65 40.64 0) (unit 1)
     (in_bom yes) (on_board yes) (dnp no) (fields_autoplaced)
@@
         (path "/7fd4875b-e2b3-49e9-a377-320ee6c6aef7/42cd8867-79f6-4c26-8217-42f6d2cc80dc"
           (reference "C31") (unit 1)
+        )
+      )
+    )
+  )
+  (symbol (lib_id "Jumper:Jumper_3_Bridged12") (at 156.21 48.26 0) (unit 1)
+    (in_bom yes) (on_board yes) (dnp no) (fields_autoplaced)
+    (property "Reference" "JP10" (at 156.21 44.3859 0)
+      (effects (font (size 1.27 1.27)))
+    )
+    (property "Value" "Jumper_3_Bridged12" (at 156.21 46.3069 0)
+      (effects (font (size 1.27 1.27)))
+    )
+    (property "Footprint" "Connector_PinHeader_2.54mm:PinHeader_1x03_P2.54mm_Vertical" (at 156.21 48.26 0)
+      (effects (font (size 1.27 1.27)) hide)
+    )
+    (property "Datasheet" "~" (at 156.21 48.26 0)
+      (effects (font (size 1.27 1.27)) hide)
+    )
+    (pin "1")
+    (pin "2")
+    (pin "3")
+    (instances
+      (project "rollo control"
+        (path "/7fd4875b-e2b3-49e9-a377-320ee6c6aef7/42cd8867-79f6-4c26-8217-42f6d2cc80dc"
+          (reference "JP10") (unit 1)
         )
       )
@@
     )
   )
-  (symbol (lib_id "Connector_Generic:Conn_01x04") (at 163.83 64.77 0) (unit 1)
-    (in_bom yes) (on_board yes) (dnp no) (fields_autoplaced)
-    (property "Reference" "UART_AUTOTERM1" (at 166.37 64.77 0)
-      (effects (font (size 1.27 1.27)) (justify left))
-    )
-    (property "Value" "Conn_01x04" (at 166.37 67.31 0)
-      (effects (font (size 1.27 1.27)) (justify left))
-    )
-    (property "Footprint" "" (at 163.83 64.77 0)
-      (effects (font (size 1.27 1.27)) hide)
-    )
-    (property "Datasheet" "~" (at 163.83 64.77 0)
-      (effects (font (size 1.27 1.27)) hide)
-    )
+  (symbol (lib_id "Connector_Generic:Conn_01x04") (at 163.83 62.23 0) (unit 1)
+    (in_bom yes) (on_board yes) (dnp no) (fields_autoplaced)
+    (property "Reference" "UART_AUTOTERM1" (at 166.37 62.23 0)
+      (effects (font (size 1.27 1.27)) (justify left))
+    )
+    (property "Value" "Conn_01x04" (at 166.37 64.77 0)
+      (effects (font (size 1.27 1.27)) (justify left))
+    )
+    (property "Footprint" "" (at 163.83 62.23 0)
+      (effects (font (size 1.27 1.27)) hide)
+    )
+    (property "Datasheet" "~" (at 163.83 62.23 0)
+      (effects (font (size 1.27 1.27)) hide)
+    )

Commit message: placing
Parts:
- removed C33: C_Small, symbol Device:C_Small
- C31, C32: footprint (none) -> Capacitor_SMD:C_0603_1608Metric_Pad1.08x0.95mm_HandSolder
- UART_AUTOTERM1: footprint (none) -> Connector_JST:JST_XH_B4B-XH-A_1x04_P2.50mm_Vertical
Changed lines of the file:
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@@
   (junction (at 114.3 38.1) (diameter 0) (color 0 0 0 0)
   )
-  (junction (at 162.56 36.83) (diameter 0) (color 0 0 0 0)
-  )
   (junction (at 137.16 69.85) (diameter 0) (color 0 0 0 0)
   )
@@
     (stroke (width 0) (type default))
   )
-  (wire (pts (xy 162.56 36.83) (xy 162.56 48.26))
-    (stroke (width 0) (type default))
-  )
-  (wire (pts (xy 173.99 36.83) (xy 173.99 38.1))
+  (wire (pts (xy 162.56 34.29) (xy 162.56 48.26))
     (stroke (width 0) (type default))
   )
@@
     (stroke (width 0) (type default))
   )
-  (wire (pts (xy 173.99 36.83) (xy 162.56 36.83))
-    (stroke (width 0) (type default))
-  )
   (wire (pts (xy 114.3 38.1) (xy 114.3 48.26))
     (stroke (width 0) (type default))
@@
   )
   (wire (pts (xy 127 64.77) (xy 142.24 64.77))
-    (stroke (width 0) (type default))
-  )
-  (wire (pts (xy 162.56 34.29) (xy 162.56 36.83))
     (stroke (width 0) (type default))
   )
@@
     (effects (font (size 1.27 1.27)) (justify left))
   )
-  (hierarchical_label "GND" (shape input) (at 173.99 43.18 270) (fields_autoplaced)
-    (effects (font (size 1.27 1.27)) (justify right))
-  )
   (hierarchical_label "GND" (shape input) (at 120.65 43.18 270) (fields_autoplaced)
     (effects (font (size 1.27 1.27)) (justify right))
   )
-  (symbol (lib_id "Device:C_Small") (at 173.99 40.64 0) (mirror y) (unit 1)
-    (in_bom yes) (on_board yes) (dnp no) (fields_autoplaced)
-    (property "Reference" "C33" (at 171.45 39.3763 0)
-      (effects (font (size 1.27 1.27)) (justify left))
-    )
-    (property "Value" "C_Small" (at 171.45 41.9163 0)
-      (effects (font (size 1.27 1.27)) (justify left))
-    )
-    (property "Footprint" "" (at 173.99 40.64 0)
-      (effects (font (size 1.27 1.27)) hide)
-    )
-    (property "Datasheet" "~" (at 173.99 40.64 0)
-      (effects (font (size 1.27 1.27)) hide)
-    )
-    (pin "1")
-    (pin "2")
-    (instances
-      (project "rollo control"
-        (path "/7fd4875b-e2b3-49e9-a377-320ee6c6aef7/42cd8867-79f6-4c26-8217-42f6d2cc80dc"
-          (reference "C33") (unit 1)
-        )
-      )
-    )
-  )
   (symbol (lib_id "Device:C_Small") (at 120.65 40.64 0) (unit 1)
     (in_bom yes) (on_board yes) (dnp no) (fields_autoplaced)
@@
       (effects (font (size 1.27 1.27)) (justify left))
     )
-    (property "Footprint" "" (at 120.65 40.64 0)
+    (property "Footprint" "Capacitor_SMD:C_0603_1608Metric_Pad1.08x0.95mm_HandSolder" (at 120.65 40.64 0)
       (effects (font (size 1.27 1.27)) hide)
     )
@@
       (effects (font (size 1.27 1.27)) (justify left))
     )
-    (property "Footprint" "" (at 163.83 62.23 0)
+    (property "Footprint" "Connector_JST:JST_XH_B4B-XH-A_1x04_P2.50mm_Vertical" (at 163.83 62.23 0)
       (effects (font (size 1.27 1.27)) hide)
     )
@@
       (effects (font (size 1.27 1.27)) (justify left))
     )
-    (property "Footprint" "" (at 134.62 54.61 0)
-      (effects (font (size 1.27 1.27)) hide)
-    )
+    (property "Footprint" "Capacitor_SMD:C_0603_1608Metric_Pad1.08x0.95mm_HandSolder" (at 134.62 54.61 0)
+      (effects (font (size 1.27 1.27)) hide)
+    )

Commit message: gsdfg
dyfg
Parts:
- removed D1: SP0502BAHT, Package_TO_SOT_SMD:SOT-23, symbol Power_Protection:SP0502BAHT
Changed lines of the file:
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@@
   (junction (at 114.3 48.26) (diameter 0) (color 0 0 0 0)
-  )
-  (junction (at 142.24 64.77) (diameter 0) (color 0 0 0 0)
-  )
-  (junction (at 139.7 90.17) (diameter 0) (color 0 0 0 0)
   )
   (junction (at 156.21 52.07) (diameter 0) (color 0 0 0 0)
@@
   (junction (at 114.3 38.1) (diameter 0) (color 0 0 0 0)
   )
-  (junction (at 137.16 69.85) (diameter 0) (color 0 0 0 0)
-  )
-  (wire (pts (xy 127 69.85) (xy 137.16 69.85))
-    (stroke (width 0) (type default))
-  )
-  (wire (pts (xy 142.24 64.77) (xy 142.24 73.66))
-    (stroke (width 0) (type default))
-  )
-  (wire (pts (xy 137.16 73.66) (xy 137.16 69.85))
+  (wire (pts (xy 127 69.85) (xy 156.21 69.85))
     (stroke (width 0) (type default))
   )
@@
     (stroke (width 0) (type default))
   )
-  (wire (pts (xy 142.24 64.77) (xy 158.75 64.77))
-    (stroke (width 0) (type default))
-  )
   (wire (pts (xy 119.38 52.07) (xy 134.62 52.07))
-    (stroke (width 0) (type default))
-  )
-  (wire (pts (xy 139.7 90.17) (xy 152.4 90.17))
     (stroke (width 0) (type default))
   )
@@
     (stroke (width 0) (type default))
   )
-  (wire (pts (xy 127 64.77) (xy 142.24 64.77))
+  (wire (pts (xy 127 64.77) (xy 158.75 64.77))
     (stroke (width 0) (type default))
   )
@@
     (stroke (width 0) (type default))
   )
-  (wire (pts (xy 139.7 83.82) (xy 139.7 90.17))
-    (stroke (width 0) (type default))
-  )
   (wire (pts (xy 114.3 34.29) (xy 114.3 38.1))
     (stroke (width 0) (type default))
   )
-  (wire (pts (xy 116.84 90.17) (xy 139.7 90.17))
-    (stroke (width 0) (type default))
-  )
-  (wire (pts (xy 156.21 69.85) (xy 137.16 69.85))
+  (wire (pts (xy 116.84 90.17) (xy 152.4 90.17))
     (stroke (width 0) (type default))
   )
@@
         )
       )
-    )
-  )
-  (symbol (lib_id "Power_Protection:SP0502BAHT") (at 139.7 78.74 0) (unit 1)
-    (in_bom yes) (on_board yes) (dnp no)
-    (property "Reference" "D1" (at 142.24 82.55 0)
-      (effects (font (size 1.27 1.27)) (justify left))
-    )
-    (property "Value" "SP0502BAHT" (at 142.24 85.09 0)
-      (effects (font (size 1.27 1.27)) (justify left))
-    )
-    (property "Footprint" "Package_TO_SOT_SMD:SOT-23" (at 145.415 80.01 0)
-      (effects (font (size 1.27 1.27)) (justify left) hide)
-    )
-    (property "Datasheet" "http://www.littelfuse.com/~/media/files/littelfuse/technical%20resources/documents/data%20sheets/sp05xxba.pdf" (at 142.875 75.565 0)
-      (effects (font (size 1.27 1.27)) hide)
-    )
-    (pin "3")
-    (pin "1")
-    (pin "2")
-    (instances
-      (project "rollo control"
-        (path "/7fd4875b-e2b3-49e9-a377-320ee6c6aef7/b6c73591-e73a-4bd7-89c6-628af8fa635f"
-          (reference "D1") (unit 1)
-        )
-        (path "/7fd4875b-e2b3-49e9-a377-320ee6c6aef7/27b75ada-6c2a-4515-886a-42a027319529"
-          (reference "D5") (unit 1)
-        )
-        (path "/7fd4875b-e2b3-49e9-a377-320ee6c6aef7/42cd8867-79f6-4c26-8217-42f6d2cc80dc"
-          (reference "D11") (unit 1)
-        )
-      )
